File: 5v_gpio.kicad_sch (KiCad schematic)
At the start: 2 parts, among them CN12 4P JST VH, CN13 4P JST VH

Commit message: Updated library name, updated and verified all footprints
Parts:
- CN12, CN13: footprint EASYEDA2KICAD:CONN-TH_B4P-VH-LF-SN -> LiveAstra:CONN-TH_B4P-VH-LF-SN; symbol EASYEDA2KICAD:JST_VH_4PIN_10A_250V -> LiveAstra:JST_VH_4PIN_10A_250V
Changed lines of the file:
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@@
 	)
 	(symbol
-		(lib_id "EASYEDA2KICAD:JST_VH_4PIN_10A_250V")
+		(lib_id "LiveAstra:JST_VH_4PIN_10A_250V")
 		(at 134.62 114.3 0)
 		(unit 1)
@@
 			)
 		)
-		(property "Footprint" "EASYEDA2KICAD:CONN-TH_B4P-VH-LF-SN"
+		(property "Footprint" "LiveAstra:CONN-TH_B4P-VH-LF-SN"
 			(at 134.62 134.62 0)
 			(effects
@@
 	)
 	(symbol
-		(lib_id "EASYEDA2KICAD:JST_VH_4PIN_10A_250V")
+		(lib_id "LiveAstra:JST_VH_4PIN_10A_250V")
 		(at 134.62 76.2 0)
 		(unit 1)
@@
 			)
 		)
-		(property "Footprint" "EASYEDA2KICAD:CONN-TH_B4P-VH-LF-SN"
+		(property "Footprint" "LiveAstra:CONN-TH_B4P-VH-LF-SN"
 			(at 134.62 96.52 0)
 			(effects
