File: amber_led_driver.kicad_sch (KiCad schematic)
At the start: 11 parts

Commit message: Updated library name, updated and verified all footprints
Parts:
- C1, C21: footprint EASYEDA2KICAD:C1206 -> LiveAstra:C1206; symbol EASYEDA2KICAD:C_10n_X7R_CERAMIC -> LiveAstra:C_10n_X7R_CERAMIC
- C2: footprint EASYEDA2KICAD:C0805 -> LiveAstra:C0805; symbol EASYEDA2KICAD:C_1uF_X7R_CERAMIC -> LiveAstra:C_1uF_X7R_CERAMIC
- C3: footprint EASYEDA2KICAD:C1206 -> LiveAstra:C1206; symbol EASYEDA2KICAD:C_22uF_X5R_CERAMIC -> LiveAstra:C_22uF_X5R_CERAMIC
- L1: footprint EASYEDA2KICAD:IND-SMD_L7.5-W7.0_SPM7054VT-330M-D -> LiveAstra:IND-SMD_L7.5-W7.0_SPM7054VT-330M-D; symbol EASYEDA2KICAD:L_4u7_7.8A_SPM7054VT-4R7M-D -> LiveAstra:L_4u7_7.8A_SPM7054VT-4R7M-D
- R1: footprint EASYEDA2KICAD:R1210 -> LiveAstra:R1210; symbol EASYEDA2KICAD:R_39mOhm_1210_500mW -> LiveAstra:R_39mOhm_1210_500mW
- U1: footprint EASYEDA2KICAD:HSOP-8_L5.0-W4.0-P1.27-LS6.2-BL-EP -> LiveAstra:HSOP-8_L5.0-W4.0-P1.27-LS6.2-BL-EP; symbol EASYEDA2KICAD:LED2001PHR -> LiveAstra:LED2001PHR
Changed lines of the file:
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@@
 	)
 	(symbol
-		(lib_id "EASYEDA2KICAD:L_4u7_7.8A_SPM7054VT-4R7M-D")
+		(lib_id "LiveAstra:L_4u7_7.8A_SPM7054VT-4R7M-D")
 		(at 166.37 78.74 0)
 		(unit 1)
@@
 			)
 		)
-		(property "Footprint" "EASYEDA2KICAD:IND-SMD_L7.5-W7.0_SPM7054VT-330M-D"
+		(property "Footprint" "LiveAstra:IND-SMD_L7.5-W7.0_SPM7054VT-330M-D"
 			(at 166.37 90.17 0)
 			(effects
@@
 	)
 	(symbol
-		(lib_id "EASYEDA2KICAD:C_10n_X7R_CERAMIC")
+		(lib_id "LiveAstra:C_10n_X7R_CERAMIC")
 		(at 177.8 86.36 90)
 		(unit 1)
@@
 			)
 		)
-		(property "Footprint" "EASYEDA2KICAD:C1206"
+		(property "Footprint" "LiveAstra:C1206"
 			(at 190.5 86.36 0)
 			(effects
@@
 	)
 	(symbol
-		(lib_id "EASYEDA2KICAD:R_39mOhm_1210_500mW")
+		(lib_id "LiveAstra:R_39mOhm_1210_500mW")
 		(at 231.14 106.68 90)
 		(unit 1)
@@
 			)
 		)
-		(property "Footprint" "EASYEDA2KICAD:R1210"
+		(property "Footprint" "LiveAstra:R1210"
 			(at 243.84 106.68 0)
 			(effects
@@
 	)
 	(symbol
-		(lib_id "EASYEDA2KICAD:C_10n_X7R_CERAMIC")
+		(lib_id "LiveAstra:C_10n_X7R_CERAMIC")
 		(at 203.2 86.36 90)
 		(unit 1)
@@
 			)
 		)
-		(property "Footprint" "EASYEDA2KICAD:C1206"
+		(property "Footprint" "LiveAstra:C1206"
 			(at 215.9 86.36 0)
 			(effects
@@
 	)
 	(symbol
-		(lib_id "EASYEDA2KICAD:LED2001PHR")
+		(lib_id "LiveAstra:LED2001PHR")
 		(at 132.08 88.9 0)
 		(unit 1)
@@
 			)
 		)
-		(property "Footprint" "EASYEDA2KICAD:HSOP-8_L5.0-W4.0-P1.27-LS6.2-BL-EP"
+		(property "Footprint" "LiveAstra:HSOP-8_L5.0-W4.0-P1.27-LS6.2-BL-EP"
 			(at 132.08 124.46 0)
 			(effects
@@
 	)
 	(symbol
-		(lib_id "EASYEDA2KICAD:C_22uF_X5R_CERAMIC")
+		(lib_id "LiveAstra:C_22uF_X5R_CERAMIC")
 		(at 50.8 86.36 90)
 		(unit 1)
@@
 			)
 		)
-		(property "Footprint" "EASYEDA2KICAD:C1206"
+		(property "Footprint" "LiveAstra:C1206"
 			(at 63.5 86.36 0)
 			(effects
@@
 	)
 	(symbol
-		(lib_id "EASYEDA2KICAD:C_1uF_X7R_CERAMIC")
+		(lib_id "LiveAstra:C_1uF_X7R_CERAMIC")
 		(at 76.2 106.68 90)
 		(unit 1)
@@
 			)
 		)
-		(property "Footprint" "EASYEDA2KICAD:C0805"
+		(property "Footprint" "LiveAstra:C0805"
 			(at 88.9 106.68 0)
 			(effects
