File: connectors.kicad_sch (KiCad schematic)
At the start: 10 parts, among them CN1 4P JST VH, CN2 4P JST VH, CN3 4P JST VH, CN4 4P JST VH, CN7 2P JST VH, CN8 2P JST VH

Commit message: Updated library name, updated and verified all footprints
Parts:
- CN1, CN2, CN3, CN4: footprint EASYEDA2KICAD:CONN-TH_B4P-VH-LF-SN -> LiveAstra:CONN-TH_B4P-VH-LF-SN; symbol EASYEDA2KICAD:JST_VH_4PIN_10A_250V -> LiveAstra:JST_VH_4PIN_10A_250V
- CN7, CN8: footprint EASYEDA2KICAD:CONN-TH_B2P-VH-R -> LiveAstra:CONN-TH_B2P-VH-R; symbol EASYEDA2KICAD:JST_VH_2PIN_10A_250V -> LiveAstra:JST_VH_2PIN_10A_250V
- D2, D3, D4, D5: footprint EASYEDA2KICAD:SMB_L4.6-W3.6-LS5.3-BI -> LiveAstra:SMB_L4.6-W3.6-LS5.3-BI; symbol EASYEDA2KICAD:D_TVS_BIDI_600W -> LiveAstra:D_TVS_BIDI_600W
Changed lines of the file:
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@@
 	)
 	(symbol
-		(lib_id "EASYEDA2KICAD:D_TVS_BIDI_600W")
+		(lib_id "LiveAstra:D_TVS_BIDI_600W")
 		(at 149.86 77.47 90)
 		(unit 1)
@@
 			)
 		)
-		(property "Footprint" "EASYEDA2KICAD:SMB_L4.6-W3.6-LS5.3-BI"
+		(property "Footprint" "LiveAstra:SMB_L4.6-W3.6-LS5.3-BI"
 			(at 158.75 77.47 0)
 			(effects
@@
 	)
 	(symbol
-		(lib_id "EASYEDA2KICAD:JST_VH_4PIN_10A_250V")
+		(lib_id "LiveAstra:JST_VH_4PIN_10A_250V")
 		(at 55.88 118.11 180)
 		(unit 1)
@@
 			)
 		)
-		(property "Footprint" "EASYEDA2KICAD:CONN-TH_B4P-VH-LF-SN"
+		(property "Footprint" "LiveAstra:CONN-TH_B4P-VH-LF-SN"
 			(at 55.88 97.79 0)
 			(effects
@@
 	)
 	(symbol
-		(lib_id "EASYEDA2KICAD:D_TVS_BIDI_600W")
+		(lib_id "LiveAstra:D_TVS_BIDI_600W")
 		(at 101.6 78.74 90)
 		(unit 1)
@@
 			)
 		)
-		(property "Footprint" "EASYEDA2KICAD:SMB_L4.6-W3.6-LS5.3-BI"
+		(property "Footprint" "LiveAstra:SMB_L4.6-W3.6-LS5.3-BI"
 			(at 110.49 78.74 0)
 			(effects
@@
 	)
 	(symbol
-		(lib_id "EASYEDA2KICAD:JST_VH_4PIN_10A_250V")
+		(lib_id "LiveAstra:JST_VH_4PIN_10A_250V")
 		(at 55.88 162.56 180)
 		(unit 1)
@@
 			)
 		)
-		(property "Footprint" "EASYEDA2KICAD:CONN-TH_B4P-VH-LF-SN"
+		(property "Footprint" "LiveAstra:CONN-TH_B4P-VH-LF-SN"
 			(at 55.88 142.24 0)
 			(effects
@@
 	)
 	(symbol
-		(lib_id "EASYEDA2KICAD:D_TVS_BIDI_600W")
+		(lib_id "LiveAstra:D_TVS_BIDI_600W")
 		(at 101.6 41.91 90)
 		(unit 1)
@@
 			)
 		)
-		(property "Footprint" "EASYEDA2KICAD:SMB_L4.6-W3.6-LS5.3-BI"
+		(property "Footprint" "LiveAstra:SMB_L4.6-W3.6-LS5.3-BI"
 			(at 110.49 41.91 0)
 			(effects
@@
 	)
 	(symbol
-		(lib_id "EASYEDA2KICAD:JST_VH_4PIN_10A_250V")
+		(lib_id "LiveAstra:JST_VH_4PIN_10A_250V")
 		(at 55.88 36.83 180)
 		(unit 1)
@@
 			)
 		)
-		(property "Footprint" "EASYEDA2KICAD:CONN-TH_B4P-VH-LF-SN"
+		(property "Footprint" "LiveAstra:CONN-TH_B4P-VH-LF-SN"
 			(at 55.88 16.51 0)
 			(effects
@@
 	)
 	(symbol
-		(lib_id "EASYEDA2KICAD:JST_VH_4PIN_10A_250V")
+		(lib_id "LiveAstra:JST_VH_4PIN_10A_250V")
 		(at 55.88 74.93 180)
 		(unit 1)
@@
 			)
 		)
-		(property "Footprint" "EASYEDA2KICAD:CONN-TH_B4P-VH-LF-SN"
+		(property "Footprint" "LiveAstra:CONN-TH_B4P-VH-LF-SN"
 			(at 55.88 54.61 0)
 			(effects
@@
 	)
 	(symbol
-		(lib_id "EASYEDA2KICAD:JST_VH_2PIN_10A_250V")
+		(lib_id "LiveAstra:JST_VH_2PIN_10A_250V")
 		(at 195.58 113.03 180)
 		(unit 1)
@@
 			)
 		)
-		(property "Footprint" "EASYEDA2KICAD:CONN-TH_B2P-VH-R"
+		(property "Footprint" "LiveAstra:CONN-TH_B2P-VH-R"
 			(at 195.58 93.98 0)
 			(effects
@@
 	)
 	(symbol
-		(lib_id "EASYEDA2KICAD:D_TVS_BIDI_600W")
+		(lib_id "LiveAstra:D_TVS_BIDI_600W")
 		(at 149.86 41.91 90)
 		(unit 1)
@@
 			)
 		)
-		(property "Footprint" "EASYEDA2KICAD:SMB_L4.6-W3.6-LS5.3-BI"
+		(property "Footprint" "LiveAstra:SMB_L4.6-W3.6-LS5.3-BI"
 			(at 158.75 41.91 0)
 			(effects
@@
 	)
 	(symbol
-		(lib_id "EASYEDA2KICAD:JST_VH_2PIN_10A_250V")
+		(lib_id "LiveAstra:JST_VH_2PIN_10A_250V")
 		(at 195.58 74.93 180)
 		(unit 1)
@@
 			)
 		)
-		(property "Footprint" "EASYEDA2KICAD:CONN-TH_B2P-VH-R"
+		(property "Footprint" "LiveAstra:CONN-TH_B2P-VH-R"
 			(at 195.58 55.88 0)
 			(effects
