File: gpio_connectors.kicad_sch (KiCad schematic)
At the start: 2 parts, among them CN11 4P JST ZH, CN12 4P JST ZH

Commit message: Updated library name, updated and verified all footprints
Parts:
- CN11, CN12: footprint EASYEDA2KICAD:CONN-TH_B4B-ZR-3.4-LF-SN -> LiveAstra:CONN-TH_B4B-ZR-3.4-LF-SN; symbol EASYEDA2KICAD:JST_ZH_4PIN_1A_50V -> LiveAstra:JST_ZH_4PIN_1A_50V
Changed lines of the file:
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@@
 	(paper "A4")
 	(symbol
-		(lib_id "EASYEDA2KICAD:JST_ZH_4PIN_1A_50V")
+		(lib_id "LiveAstra:JST_ZH_4PIN_1A_50V")
 		(at 137.16 73.66 180)
 		(unit 1)
@@
 			)
 		)
-		(property "Footprint" "EASYEDA2KICAD:CONN-TH_B4B-ZR-3.4-LF-SN"
+		(property "Footprint" "LiveAstra:CONN-TH_B4B-ZR-3.4-LF-SN"
 			(at 137.16 57.15 0)
 			(effects
@@
 	)
 	(symbol
-		(lib_id "EASYEDA2KICAD:JST_ZH_4PIN_1A_50V")
+		(lib_id "LiveAstra:JST_ZH_4PIN_1A_50V")
 		(at 137.16 111.76 180)
 		(unit 1)
@@
 			)
 		)
-		(property "Footprint" "EASYEDA2KICAD:CONN-TH_B4B-ZR-3.4-LF-SN"
+		(property "Footprint" "LiveAstra:CONN-TH_B4B-ZR-3.4-LF-SN"
 			(at 137.16 95.25 0)
 			(effects
