File: led_connectors.kicad_sch (KiCad schematic)
At the start: 2 parts, among them CN14 4P JST ZH, CN20 4P JST ZH

Commit message: Updated library name, updated and verified all footprints
Parts:
- CN14, CN20: footprint EASYEDA2KICAD:CONN-TH_B4B-ZR-3.4-LF-SN -> LiveAstra:CONN-TH_B4B-ZR-3.4-LF-SN; symbol EASYEDA2KICAD:JST_ZH_4PIN_1A_50V -> LiveAstra:JST_ZH_4PIN_1A_50V
Changed lines of the file:
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@@
 	)
 	(symbol
-		(lib_id "EASYEDA2KICAD:JST_ZH_4PIN_1A_50V")
+		(lib_id "LiveAstra:JST_ZH_4PIN_1A_50V")
 		(at 193.1505 86.4569 0)
 		(unit 1)
@@
 			)
 		)
-		(property "Footprint" "EASYEDA2KICAD:CONN-TH_B4B-ZR-3.4-LF-SN"
+		(property "Footprint" "LiveAstra:CONN-TH_B4B-ZR-3.4-LF-SN"
 			(at 193.1505 102.9669 0)
 			(effects
@@
 	)
 	(symbol
-		(lib_id "EASYEDA2KICAD:JST_ZH_4PIN_1A_50V")
+		(lib_id "LiveAstra:JST_ZH_4PIN_1A_50V")
 		(at 199.39 129.54 0)
 		(unit 1)
@@
 			)
 		)
-		(property "Footprint" "EASYEDA2KICAD:CONN-TH_B4B-ZR-3.4-LF-SN"
+		(property "Footprint" "LiveAstra:CONN-TH_B4B-ZR-3.4-LF-SN"
 			(at 199.39 146.05 0)
 			(effects
