File: led_pwm_connectors.kicad_sch (KiCad schematic)
At the start: 2 parts, among them CN2 JST_VH_8PIN_10A_250V

Commit message: Updated library name, updated and verified all footprints
Parts:
- CN2: footprint easyeda2kicad:CONN-TH_B8P-VH-B-LF-SN -> LiveAstra:CONN-TH_B8P-VH-B-LF-SN; symbol EASYEDA2KICAD:JST_VH_8PIN_10A_250V -> LiveAstra:JST_VH_8PIN_10A_250V
- R34: symbol EASYEDA2KICAD:R_0Ohm_0805_125mW -> LiveAstra:R_0Ohm_0805_125mW
Changed lines of the file:
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@@
 	)
 	(symbol
-		(lib_id "EASYEDA2KICAD:JST_VH_8PIN_10A_250V")
+		(lib_id "LiveAstra:JST_VH_8PIN_10A_250V")
 		(at 182.88 96.52 0)
 		(unit 1)
@@
 			)
 		)
-		(property "Footprint" "easyeda2kicad:CONN-TH_B8P-VH-B-LF-SN"
+		(property "Footprint" "LiveAstra:CONN-TH_B8P-VH-B-LF-SN"
 			(at 182.88 129.54 0)
 			(effects
@@
 	)
 	(symbol
-		(lib_id "EASYEDA2KICAD:+5V_IN")
+		(lib_id "LiveAstra:+5V_IN")
 		(at 167.64 124.46 0)
 		(unit 1)
@@
 	)
 	(symbol
-		(lib_id "EASYEDA2KICAD:R_0Ohm_0805_125mW")
+		(lib_id "LiveAstra:R_0Ohm_0805_125mW")
 		(at 144.78 104.14 0)
 		(unit 1)
