File: AstraControl.kicad_pcb (KiCad board)
At the start: 4 copper layers, 102 x 96 mm, 152 parts, among them CN1 4P JST VH, CN10 JST_ZH_6PIN_1A_250V, CN2 4P JST VH, CN3 4P JST VH, CN4 4P JST ZH, CN5 4P JST ZH, CN6 4P JST ZH, CN7 JST_VH_8PIN_10A_250V, CN8 4P JST ZH, CN9 4P JST ZH, SW1 TS_Basic_Small, SW2 TS_Basic_Small, U1 ESP32-S3-WROOM-1U-N8, U2 NCP361SNT1G, U3 ST1S12GR, U4 SN65HVD1782DR, U6 TXB0104PWR, U7 USBLC6-2SC6

Commit message: Ready for kibot
Parts:
- moved C25 3.08 mm to (199.8, 82.8), turned to -90 degrees
- moved R37 1.25 mm to (199.8, 77.8), turned to 90 degrees
Connections:
- net /Block Diagram/Button, Status LED, UART and I2S/GPIO_12_BUTTON renamed /Block Diagram/Button, Status LED, UART and I2S/BUTTON
- net /Block Diagram/Button, Status LED, UART and I2S/GPIO_12_BUTTON_0 renamed /Block Diagram/Button, Status LED, UART and I2S/BUTTON_0
- net /Block Diagram/Button, Status LED, UART and I2S/GPIO_12_BUTTON_CONN renamed /Block Diagram/Button, Status LED, UART and I2S/BUTTON_CONN
- net /Block Diagram/Button, Status LED, UART and I2S/GPIO_13_STATUS_LED renamed /Block Diagram/Button, Status LED, UART and I2S/STATUS_LED
- net /Block Diagram/Button, Status LED, UART and I2S/GPIO_13_STATUS_LED_CONN renamed /Block Diagram/Button, Status LED, UART and I2S/STATUS_LED_CONN
- net /Block Diagram/Button, Status LED, UART and I2S/GPIO_14_I2S_WS renamed /Block Diagram/Button, Status LED, UART and I2S/I2S_WS
- net /Block Diagram/Button, Status LED, UART and I2S/GPIO_21_I2S_SCK renamed /Block Diagram/Button, Status LED, UART and I2S/I2S_SCK
- net /Block Diagram/Button, Status LED, UART and I2S/GPIO_47_I2S_SD renamed /Block Diagram/Button, Status LED, UART and I2S/I2S_SD
- net /Block Diagram/Button, Status LED, UART and I2S/GPIO_48_I2S_LR renamed /Block Diagram/Button, Status LED, UART and I2S/I2S_LR
- net /Block Diagram/LED PWM Connector/GPIO_39_PWM_CH1 renamed /Block Diagram/LED PWM Connector/PWM_CH4
- net /Block Diagram/LED PWM Connector/GPIO_40_PWM_CH2 renamed /Block Diagram/LED PWM Connector/PWM_CH1
- net /Block Diagram/LED PWM Connector/GPIO_41_PWM_CH3 renamed /Block Diagram/LED PWM Connector/PWM_CH2
- net /Block Diagram/LED PWM Connector/GPIO_42_PWM_CH4 renamed /Block Diagram/LED PWM Connector/PWM_CH3
- net /Block Diagram/LED PWM Connector/LED_GPIO_39_CONN renamed /Block Diagram/LED PWM Connector/PWM_CH4_CONN
- net /Block Diagram/LED PWM Connector/LED_GPIO_40_CONN renamed /Block Diagram/LED PWM Connector/PWM_CH1_CONN
- net /Block Diagram/LED PWM Connector/LED_GPIO_42_CONN renamed /Block Diagram/LED PWM Connector/PWM_CH3_CONN
- net /Block Diagram/LED PWM Connector/LED_GPIO_43_CONN renamed /Block Diagram/LED PWM Connector/PWM_CH2_CONN
- net /Block Diagram/LED PWM Connector/LED_GPIO_OR_GND_CONN renamed /Block Diagram/LED PWM Connector/LED_EXTRA_PIN
- net /Block Diagram/MCU/GPIO_15_RS485_DE renamed /Block Diagram/MCU/GPIO_5_RS485_DE
- net /Block Diagram/MCU/GPIO_15_RS485_RE renamed /Block Diagram/MCU/GPIO_6_RS485_RE
- net /Block Diagram/MCU/GPIO_17_RS485_TX renamed /Block Diagram/MCU/GPIO_4_RS485_TX
- net /Block Diagram/MCU/GPIO_18_RS485_RX renamed /Block Diagram/MCU/GPIO_7_RS485_RX
- net /Block Diagram/MCU/IO2_DEBUG_LED renamed /Block Diagram/MCU/GPIO_2_DEBUG_LED
- net /Block Diagram/MCU/IO2_DEBUG_LED_CL renamed /Block Diagram/MCU/GPIO_2_DEBUG_LED_CL
Routing:
- net GND: vias 301 -> 299
Other:
- board text added: "15"
- board text added: "16"
- board text added: "17"
- board text added: "18"
- board text added: "3V3"
- board text added: "5V"
- board text added: "5V IN"
- board text added: "A"
- board text added: "B"
- board text added: "BTN"
- board text added: "D+"
- board text added: "D-"
- board text added: "DE"
- board text added: "EN"
- board text added: "FAN"
- board text added: "G"
- board text added: "GND"
- board text added: "IO0"
- board text added: "IO15"
- board text added: "IO16"
- board text added: "IO17"
- board text added: "IO18"
- board text added: "IO3"
- board text added: "IO39"
- board text added: "IO40"
- board text added: "IO41"
- board text added: "IO42"
- board text added: "LED"
- board text added: "LR"
- board text added: "OE"
- board text added: "RE"
- board text added: "RESET"
- board text added: "RX"
- board text added: "SCK"
- board text added: "SCL"
- board text added: "SD"
- board text added: "SDA"
- board text added: "TCH"
- board text added: "TX"
- board text added: "VBUS"
- board text added: "WS"
- board text added: "[ ]"
- board text added: "~3V3"
