File: AstraControl.kicad_pcb (KiCad board)
At the start: 4 copper layers, 102 x 96 mm, 152 parts, among them CN1 4P JST VH, CN10 JST_ZH_6PIN_1A_250V, CN2 4P JST VH, CN3 4P JST VH, CN4 4P JST ZH, CN5 4P JST ZH, CN6 4P JST ZH, CN7 JST_VH_8PIN_10A_250V, CN8 4P JST ZH, CN9 4P JST ZH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

Commit message: workflow
Routing:
- net GND: track 81.6 -> 81.4 mm, vias 299 -> 293
