File: mcu_power_supply.kicad_sch (KiCad schematic)
At the start: 13 parts, among them U4 NCP361SNT1G

Commit message: Updated library name, updated and verified all footprints
Parts:
- C12, C13: footprint EASYEDA2KICAD:C0402 -> LiveAstra:C0402; symbol EASYEDA2KICAD:C_1uF_X5R_0402 -> LiveAstra:C_1uF_X5R_0402
- D5: footprint easyeda2kicad:SMA_L4.2-W2.6-LS5.3-RD -> LiveAstra:SMA_L4.2-W2.6-LS5.3-RD; symbol EASYEDA2KICAD:D_Schottky_1A_40V -> LiveAstra:D_Schottky_1A_40V
- LED1: footprint EASYEDA2KICAD:LED0603-RD -> LiveAstra:LED0603-RD; symbol EASYEDA2KICAD:LED_RED_20mA_0603 -> LiveAstra:LED_RED_20mA_0603
- R7: footprint EASYEDA2KICAD:R0402 -> LiveAstra:R0402; symbol EASYEDA2KICAD:R_1MOhm_0402_62mW -> LiveAstra:R_1MOhm_0402_62mW
- R8: footprint EASYEDA2KICAD:R0402 -> LiveAstra:R0402; symbol EASYEDA2KICAD:R_220Ohm_0402_62mW -> LiveAstra:R_220Ohm_0402_62mW
- U4: footprint EASYEDA2KICAD:TSOP-5_L3.0-W1.5-P0.95-BL -> LiveAstra:TSOP-5_L3.0-W1.5-P0.95-BL; symbol EASYEDA2KICAD:U_5V_Protection_IC_TSOP -> LiveAstra:U_5V_Protection_IC_TSOP
Changed lines of the file:
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@@
 	)
 	(symbol
-		(lib_id "EASYEDA2KICAD:C_1uF_X5R_0402")
+		(lib_id "LiveAstra:C_1uF_X5R_0402")
 		(at 127 90.17 90)
 		(unit 1)
@@
 			)
 		)
-		(property "Footprint" "EASYEDA2KICAD:C0402"
+		(property "Footprint" "LiveAstra:C0402"
 			(at 139.7 90.17 0)
 			(effects
@@
 	)
 	(symbol
-		(lib_id "EASYEDA2KICAD:LED_RED_20mA_0603")
+		(lib_id "LiveAstra:LED_RED_20mA_0603")
 		(at 201.93 90.17 270)
 		(unit 1)
@@
 			)
 		)
-		(property "Footprint" "EASYEDA2KICAD:LED0603-RD"
+		(property "Footprint" "LiveAstra:LED0603-RD"
 			(at 189.23 90.17 0)
 			(effects
@@
 	)
 	(symbol
-		(lib_id "EASYEDA2KICAD:R_220Ohm_0402_62mW")
+		(lib_id "LiveAstra:R_220Ohm_0402_62mW")
 		(at 201.93 101.6 270)
 		(unit 1)
@@
 			)
 		)
-		(property "Footprint" "EASYEDA2KICAD:R0402"
+		(property "Footprint" "LiveAstra:R0402"
 			(at 193.04 101.6 0)
 			(effects
@@
 	)
 	(symbol
-		(lib_id "EASYEDA2KICAD:R_1MOhm_0402_62mW")
+		(lib_id "LiveAstra:R_1MOhm_0402_62mW")
 		(at 119.38 109.22 180)
 		(unit 1)
@@
 			)
 		)
-		(property "Footprint" "EASYEDA2KICAD:R0402"
+		(property "Footprint" "LiveAstra:R0402"
 			(at 119.38 92.71 0)
 			(effects
@@
 	)
 	(symbol
-		(lib_id "EASYEDA2KICAD:D_Schottky_1A_40V")
+		(lib_id "LiveAstra:D_Schottky_1A_40V")
 		(at 86.36 100.33 180)
 		(unit 1)
@@
 			)
 		)
-		(property "Footprint" "easyeda2kicad:SMA_L4.2-W2.6-LS5.3-RD"
+		(property "Footprint" "LiveAstra:SMA_L4.2-W2.6-LS5.3-RD"
 			(at 86.36 91.44 0)
 			(effects
@@
 	)
 	(symbol
-		(lib_id "EASYEDA2KICAD:U_5V_Protection_IC_TSOP")
+		(lib_id "LiveAstra:U_5V_Protection_IC_TSOP")
 		(at 152.4 101.6 0)
 		(unit 1)
@@
 			)
 		)
-		(property "Footprint" "EASYEDA2KICAD:TSOP-5_L3.0-W1.5-P0.95-BL"
+		(property "Footprint" "LiveAstra:TSOP-5_L3.0-W1.5-P0.95-BL"
 			(at 152.4 142.24 0)
 			(effects
@@
 	)
 	(symbol
-		(lib_id "EASYEDA2KICAD:C_1uF_X5R_0402")
+		(lib_id "LiveAstra:C_1uF_X5R_0402")
 		(at 168.91 90.17 270)
 		(unit 1)
@@
 			)
 		)
-		(property "Footprint" "EASYEDA2KICAD:C0402"
+		(property "Footprint" "LiveAstra:C0402"
 			(at 156.21 90.17 0)
 			(effects

Commit message: Work on kibot
Changed lines of the file:
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@@
-		)
-	)
-	(polyline
-		(pts
-			(xy 131.1298 46.6355) (xy 131.1428 46.6365) (xy 131.1557 46.6381) (xy 131.1685 46.6403) (xy 131.1812 46.6432)
-			(xy 131.1936 46.6466) (xy 131.2059 46.6507) (xy 131.2179 46.6553) (xy 131.2297 46.6606) (xy 131.2413 46.6664)
-			(xy 131.2525 46.6727) (xy 131.2635 46.6797) (xy 131.2741 46.6871) (xy 131.2843 46.6951) (xy 131.2942 46.7037)
-			(xy 131.3038 46.7127) (xy 131.3128 46.7222) (xy 131.3213 46.7321) (xy 131.3293 46.7424) (xy 131.3368 46.753)
-			(xy 131.3437 46.7639) (xy 131.3501 46.7752) (xy 131.3559 46.7867) (xy 131.3611 46.7985) (xy 131.3658 46.8106)
-			(xy 131.3698 46.8228) (xy 131.3733 46.8353) (xy 131.3761 46.8479) (xy 131.3784 46.8607) (xy 131.38 46.8736)
-			(xy 131.3809 46.8867) (xy 131.3812 46.8998) (xy 131.3812 48.355) (xy 131.6458 48.355) (xy 131.6458 48.6196)
-			(xy 130.8521 48.6196) (xy 130.8521 48.355) (xy 131.1167 48.355) (xy 131.1167 46.8998) (xy 130.7198 46.8998)
-			(xy 130.7198 46.6352) (xy 131.1167 46.6352) (xy 131.1298 46.6355)
-		)
-		(stroke
-			(width -0.0001)
-			(type solid)
-		)
-		(fill
-			(type color)
-			(color 34 187 51 1)
-		)
-	)
-	(polyline
-		(pts
-			(xy 131.2216 45.1826) (xy 131.3259 45.1904) (xy 131.4292 45.2032) (xy 131.5315 45.221) (xy 131.6326 45.2438)
-			(xy 131.7323 45.2715) (xy 131.8304 45.3039) (xy 131.9267 45.3411) (xy 132.0211 45.3829) (xy 132.1134 45.4294)
-			(xy 132.2034 45.4803) (xy 132.291 45.5356) (xy 132.376 45.5953) (xy 132.4581 45.6593) (xy 132.5373 45.7276)
-			(xy 132.6134 45.8) (xy 132.6858 45.876) (xy 132.754 45.9552) (xy 132.818 46.0374) (xy 132.8777 46.1223)
-			(xy 132.9331 46.2099) (xy 132.984 46.2999) (xy 133.0304 46.3923) (xy 133.0722 46.4867) (xy 133.1094 46.583)
-			(xy 133.1418 46.6811) (xy 133.1695 46.7807) (xy 133.1923 46.8818) (xy 133.2101 46.9841) (xy 133.223 47.0875)
-			(xy 133.2307 47.1917) (xy 133.2333 47.2967) (xy 133.2318 47.3767) (xy 133.2273 47.4561) (xy 133.2199 47.5349)
-			(xy 133.2096 47.6131) (xy 133.1965 47.6904) (xy 133.1805 47.767) (xy 133.1618 47.8426) (xy 133.1404 47.9173)
-			(xy 133.1163 47.991) (xy 133.0896 48.0636) (xy 133.0603 48.135) (xy 133.0284 48.2052) (xy 132.9941 48.2742)
-			(xy 132.9573 48.3418) (xy 132.9182 48.4079) (xy 132.8766 48.4726) (xy 132.8327 48.5358) (xy 132.7866 48.5973)
-			(xy 132.7382 48.6571) (xy 132.6877 48.7152) (xy 132.635 48.7715) (xy 132.5802 48.8259) (xy 132.5234 48.8784)
-			(xy 132.4645 48.9288) (xy 132.4037 48.9772) (xy 132.341 49.0234) (xy 132.2764 49.0675) (xy 132.2099 49.1092)
-			(xy 132.1417 49.1487) (xy 132.0717 49.1857) (xy 132 49.2202) (xy 131.9267 49.2522) (xy 131.7771 49.3077)
-			(xy 131.6253 49.3514) (xy 131.472 49.3834) (xy 131.3177 49.4039) (xy 131.1631 49.4129) (xy 131.0089 49.4106)
-			(xy 130.8555 49.3972) (xy 130.7037 49.3727) (xy 130.5541 49.3372) (xy 130.4073 49.291) (xy 130.2639 49.234)
-			(xy 130.1245 49.1665) (xy 129.9898 49.0886) (xy 129.8604 49.0003) (xy 129.7369 48.9019) (xy 129.62 48.7934)
-			(xy 129.5114 48.6764) (xy 129.413 48.5529) (xy 129.3247 48.4235) (xy 129.2468 48.2888) (xy 129.1793 48.1494)
-			(xy 129.1224 48.006) (xy 129.0761 47.8592) (xy 129.0407 47.7096) (xy 129.0162 47.5578) (xy 129.0027 47.4045)
-			(xy 129.0017 47.3373) (xy 129.265 47.3373) (xy 129.2729 47.4726) (xy 129.2908 47.6076) (xy 129.3188 47.7417)
-			(xy 129.357 47.8745) (xy 129.4056 48.0054) (xy 129.4638 48.1323) (xy 129.5307 48.2533) (xy 129.6057 48.3679)
-			(xy 129.6885 48.476) (xy 129.7786 48.5773) (xy 129.8754 48.6713) (xy 129.9786 48.7579) (xy 130.0877 48.8366)
-			(xy 130.2022 48.9073) (xy 130.3217 48.9695) (xy 130.4456 49.023) (xy 130.5736 49.0674) (xy 130.7052 49.1025)
-			(xy 130.8398 49.128) (xy 130.9772 49.1435) (xy 131.1167 49.1487) (xy 131.2085 49.1465) (xy 131.2997 49.1397)
-			(xy 131.3902 49.1285) (xy 131.4797 49.1128) (xy 131.5681 49.0929) (xy 131.6553 49.0687) (xy 131.7411 49.0403)
-			(xy 131.8254 49.0078) (xy 131.908 48.9712) (xy 131.9888 48.9306) (xy 132.0676 48.886) (xy 132.1442 48.8376)
-			(xy 132.2185 48.7853) (xy 132.2904 48.7293) (xy 132.3597 48.6696) (xy 132.4263 48.6063) (xy 132.4896 48.5397)
-			(xy 132.5493 48.4704) (xy 132.6053 48.3985) (xy 132.6576 48.3242) (xy 132.706 48.2476) (xy 132.7506 48.1688)
-			(xy 132.7912 48.088) (xy 132.8278 48.0054) (xy 132.8603 47.9211) (xy 132.8887 47.8353) (xy 132.9129 47.7481)
-			(xy 132.9328 47.6597) (xy 132.9485 47.5702) (xy 132.9597 47.4797) (xy 132.9665 47.3885) (xy 132.9687 47.2967)
-			(xy 132.9674 47.2267) (xy 132.9635 47.1572) (xy 132.957 47.0882) (xy 132.948 47.0198) (xy 132.9365 46.9521)
-			(xy 132.9225 46.8852) (xy 132.9062 46.819) (xy 132.8874 46.7536) (xy 132.8663 46.6891) (xy 132.843 46.6256)
-			(xy 132.8173 46.5631) (xy 132.7895 46.5017) (xy 132.7594 46.4413) (xy 132.7273 46.3822) (xy 132.693 46.3243)
-			(xy 132.6566 46.2677) (xy 132.6182 46.2125) (xy 132.5779 46.1586) (xy 132.5355 46.1063) (xy 132.4913 46.0554)
-			(xy 132.4452 46.0062) (xy 132.3973 45.9586) (xy 132.3475 45.9127) (xy 132.296 45.8685) (xy 132.2428 45.8262)
-			(xy 132.1879 45.7857) (xy 132.1314 45.7472) (xy 132.0733 45.7107) (xy 132.0136 45.6762) (xy 131.9523 45.6438)
-			(xy 131.8896 45.6136) (xy 131.8254 45.5856) (xy 131.6945 45.537) (xy 131.5617 45.4988) (xy 131.4276 45.4708)
-			(xy 131.2926 45.4529) (xy 131.1573 45.445) (xy 131.0223 45.447) (xy 130.8882 45.4587) (xy 130.7553 45.4802)
-			(xy 130.6244 45.5112) (xy 130.496 45.5517) (xy 130.3705 45.6015) (xy 130.2486 45.6605) (xy 130.1307 45.7287)
-			(xy 130.0175 45.806) (xy 129.9094 45.8921) (xy 129.807 45.987) (xy 129.7121 46.0894) (xy 129.626 46.1975)
-			(xy 129.5487 46.3107) (xy 129.4805 46.4286) (xy 129.4215 46.5505) (xy 129.3717 46.676) (xy 129.3312 46.8044)
-			(xy 129.3002 46.9353) (xy 129.2787 47.0682) (xy 129.267 47.2023) (xy 129.265 47.3373) (xy 129.0017 47.3373)
-			(xy 129.0004 47.2502) (xy 129.0095 47.0956) (xy 129.0299 46.9414) (xy 129.0619 46.788) (xy 129.1056 46.6363)
-			(xy 129.1611 46.4867) (xy 129.2277 46.3416) (xy 129.3041 46.2034) (xy 129.3899 46.0724) (xy 129.4845 45.9488)
-			(xy 129.5874 45.8331) (xy 129.6981 45.7256) (xy 129.816 45.6267) (xy 129.9407 45.5367) (xy 130.0716 45.456)
-			(xy 130.2081 45.3849) (xy 130.3497 45.3237) (xy 130.496 45.2729) (xy 130.6464 45.2328) (xy 130.8003 45.2037)
-			(xy 130.9572 45.186) (xy 131.1167 45.18) (xy 131.2216 45.1826)
-		)
-		(stroke
-			(width -0.0001)
-			(type solid)
-		)
-		(fill
-			(type color)
-			(color 34 187 51 1)
-		)
-	)
-	(polyline
-		(pts
-			(xy 131.1303 45.8418) (xy 131.1437 45.8428) (xy 131.157 45.8445) (xy 131.17 45.8468) (xy 131.1828 45.8498)
-			(xy 131.1953 45.8534) (xy 131.2076 45.8575) (xy 131.2197 45.8623) (xy 131.2314 45.8675) (xy 131.2428 45.8734)
-			(xy 131.2539 45.8798) (xy 131.2646 45.8866) (xy 131.275 45.894) (xy 131.285 45.9019) (xy 131.2946 45.9102)
-			(xy 131.3038 45.919) (xy 131.3125 45.9281) (xy 131.3208 45.9377) (xy 131.3287 45.9477) (xy 131.3361 45.9581)
-			(xy 131.3429 45.9688) (xy 131.3493 45.9799) (xy 131.3552 45.9913) (xy 131.3605 46.0031) (xy 131.3652 46.0151)
-			(xy 131.3694 46.0274) (xy 131.3729 46.0399) (xy 131.3759 46.0527) (xy 131.3782 46.0657) (xy 131.3799 46.079)
-			(xy 131.3809 46.0924) (xy 131.3812 46.106) (xy 131.3809 46.1197) (xy 131.3799 46.1331) (xy 131.3782 46.1463)
-			(xy 131.3759 46.1594) (xy 131.3729 46.1722) (xy 131.3694 46.1847) (xy 131.3652 46.197) (xy 131.3605 46.209)
-			(xy 131.3552 46.2207) (xy 131.3493 46.2322) (xy 131.3429 46.2432) (xy 131.3361 46.254) (xy 131.3287 46.2643)
-			(xy 131.3208 46.2743) (xy 131.3125 46.2839) (xy 131.3038 46.2931) (xy 131.2946 46.3019) (xy 131.285 46.3102)
-			(xy 131.275 46.3181) (xy 131.2646 46.3254) (xy 131.2539 46.3323) (xy 131.2428 46.3387) (xy 131.2314 46.3445)
-			(xy 131.2197 46.3498) (xy 131.2076 46.3546) (xy 131.1953 46.3587) (xy 131.1828 46.3623) (xy 131.17 46.3652)
-			(xy 131.157 46.3676) (xy 131.1437 46.3693) (xy 131.1303 46.3703) (xy 131.1167 46.3706) (xy 131.1031 46.3703)
-			(xy 131.0896 46.3693) (xy 131.0764 46.3676) (xy 131.0633 46.3652) (xy 131.0505 46.3623) (xy 131.038 46.3587)
-			(xy 131.0257 46.3546) (xy 131.0137 46.3498) (xy 131.002 46.3445) (xy 130.9906 46.3387) (xy 130.9795 46.3323)
-			(xy 130.9687 46.3254) (xy 130.9584 46.3181) (xy 130.9484 46.3102) (xy 130.9388 46.3019) (xy 130.9296 46.2931)
-			(xy 130.9208 46.2839) (xy 130.9125 46.2743) (xy 130.9046 46.2643) (xy 130.8973 46.254) (xy 130.8904 46.2432)
-			(xy 130.884 46.2322) (xy 130.8782 46.2207) (xy 130.8729 46.209) (xy 130.8681 46.197) (xy 130.864 46.1847)
-			(xy 130.8604 46.1722) (xy 130.8575 46.1594) (xy 130.8551 46.1463) (xy 130.8534 46.1331) (xy 130.8524 46.1197)
-			(xy 130.8521 46.106) (xy 130.8524 46.0924) (xy 130.8534 46.079) (xy 130.8551 46.0657) (xy 130.8575 46.0527)
-			(xy 130.8604 46.0399) (xy 130.864 46.0274) (xy 130.8681 46.0151) (xy 130.8729 46.0031) (xy 130.8782 45.9913)
-			(xy 130.884 45.9799) (xy 130.8904 45.9688) (xy 130.8973 45.9581) (xy 130.9046 45.9477) (xy 130.9125 45.9377)
-			(xy 130.9208 45.9281) (xy 130.9296 45.919) (xy 130.9388 45.9102) (xy 130.9484 45.9019) (xy 130.9584 45.894)
-			(xy 130.9687 45.8866) (xy 130.9795 45.8798) (xy 130.9906 45.8734) (xy 131.002 45.8675) (xy 131.0137 45.8623)
-			(xy 131.0257 45.8575) (xy 131.038 45.8534) (xy 131.0505 45.8498) (xy 131.0633 45.8468) (xy 131.0764 45.8445)
-			(xy 131.0896 45.8428) (xy 131.1031 45.8418) (xy 131.1167 45.8415) (xy 131.1303 45.8418)
-		)
-		(stroke
-			(width -0.0001)
-			(type solid)
-		)
-		(fill
-			(type color)
-			(color 34 187 51 1)
 		)
 	)
