File: 3v3_to_5v_logic_shifter.kicad_sch (KiCad schematic)
At the start: 17 parts, among them U6 TXB0104PWR

Commit message: Updated library name, updated and verified all footprints
Parts:
- C19, C20: symbol EASYEDA2KICAD:C_100nF_X7R_0402 -> LiveAstra:C_100nF_X7R_0402
- R21: symbol EASYEDA2KICAD:R_0Ohm_0805_125mW -> LiveAstra:R_0Ohm_0805_125mW
- R22: symbol EASYEDA2KICAD:R_10kOhm_0402_62mW -> LiveAstra:R_10kOhm_0402_62mW
- TP36, TP37, TP38, TP39, TP40, TP41, TP42, TP43, TP44, TP45, TP46, TP47: symbol EASYEDA2KICAD:TestPoint_Thimble -> LiveAstra:TestPoint_Thimble
- U6: footprint EASYEDA2KICAD:TSSOP-14_L5.0-W4.4-P0.65-LS6.4-BL -> LiveAstra:LOGIC_SHIFTER_TXB0104PWR_TSOP_14; symbol EASYEDA2KICAD:U_TXB0104PWR_4Bit_Logic_Level_Translator -> LiveAstra:U_TXB0104PWR_4Bit_Logic_Level_Translator
Changed lines of the file:
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@@
 	)
 	(symbol
-		(lib_id "EASYEDA2KICAD:TestPoint_Thimble")
+		(lib_id "LiveAstra:TestPoint_Thimble")
 		(at 177.8 137.16 0)
 		(unit 1)
@@
 	)
 	(symbol
-		(lib_id "EASYEDA2KICAD:TestPoint_Thimble")
+		(lib_id "LiveAstra:TestPoint_Thimble")
 		(at 129.54 91.44 0)
 		(unit 1)
@@
 	)
 	(symbol
-		(lib_id "EASYEDA2KICAD:R_10kOhm_0402_62mW")
+		(lib_id "LiveAstra:R_10kOhm_0402_62mW")
 		(at 106.68 83.82 90)
 		(unit 1)
@@
 	)
 	(symbol
-		(lib_id "EASYEDA2KICAD:TestPoint_Thimble")
+		(lib_id "LiveAstra:TestPoint_Thimble")
 		(at 129.54 106.68 0)
 		(unit 1)
@@
 	)
 	(symbol
-		(lib_id "EASYEDA2KICAD:TestPoint_Thimble")
+		(lib_id "LiveAstra:TestPoint_Thimble")
 		(at 81.28 116.84 0)
 		(unit 1)
@@
 	)
 	(symbol
-		(lib_id "EASYEDA2KICAD:U_TXB0104PWR_4Bit_Logic_Level_Translator")
+		(lib_id "LiveAstra:U_TXB0104PWR_4Bit_Logic_Level_Translator")
 		(at 152.4 88.9 0)
 		(unit 1)
@@
 			)
 		)
-		(property "Footprint" "EASYEDA2KICAD:TSSOP-14_L5.0-W4.4-P0.65-LS6.4-BL"
+		(property "Footprint" "LiveAstra:LOGIC_SHIFTER_TXB0104PWR_TSOP_14"
 			(at 153.67 148.59 0)
 			(effects
@@
 	)
 	(symbol
-		(lib_id "EASYEDA2KICAD:TestPoint_Thimble")
+		(lib_id "LiveAstra:TestPoint_Thimble")
 		(at 215.9 116.84 0)
 		(unit 1)
@@
 	)
 	(symbol
-		(lib_id "EASYEDA2KICAD:TestPoint_Thimble")
+		(lib_id "LiveAstra:TestPoint_Thimble")
 		(at 106.68 111.76 0)
 		(unit 1)
@@
 	)
 	(symbol
-		(lib_id "EASYEDA2KICAD:R_0Ohm_0805_125mW")
+		(lib_id "LiveAstra:R_0Ohm_0805_125mW")
 		(at 88.9 76.2 0)
 		(unit 1)
@@
 	)
 	(symbol
-		(lib_id "EASYEDA2KICAD:TestPoint_Thimble")
+		(lib_id "LiveAstra:TestPoint_Thimble")
 		(at 167.64 106.68 0)
 		(unit 1)
@@
 	)
 	(symbol
-		(lib_id "EASYEDA2KICAD:TestPoint_Thimble")
+		(lib_id "LiveAstra:TestPoint_Thimble")
 		(at 55.88 121.92 0)
 		(unit 1)
@@
 	)
 	(symbol
-		(lib_id "EASYEDA2KICAD:TestPoint_Thimble")
+		(lib_id "LiveAstra:TestPoint_Thimble")
 		(at 243.84 121.92 0)
 		(unit 1)
@@
 	)
 	(symbol
-		(lib_id "EASYEDA2KICAD:TestPoint_Thimble")
+		(lib_id "LiveAstra:TestPoint_Thimble")
 		(at 177.8 48.26 0)
 		(unit 1)
@@
 	)
 	(symbol
-		(lib_id "EASYEDA2KICAD:C_100nF_X7R_0402")
+		(lib_id "LiveAstra:C_100nF_X7R_0402")
 		(at 114.3 58.42 90)
 		(unit 1)
@@
 	)
 	(symbol
-		(lib_id "EASYEDA2KICAD:C_100nF_X7R_0402")
+		(lib_id "LiveAstra:C_100nF_X7R_0402")
 		(at 190.5 58.42 90)
 		(unit 1)
@@
 	)
 	(symbol
-		(lib_id "EASYEDA2KICAD:TestPoint_Thimble")
+		(lib_id "LiveAstra:TestPoint_Thimble")
 		(at 127 48.26 0)
 		(unit 1)
@@
 	)
 	(symbol
-		(lib_id "EASYEDA2KICAD:TestPoint_Thimble")
+		(lib_id "LiveAstra:TestPoint_Thimble")
 		(at 190.5 111.76 0)
 		(unit 1)

Commit message: Finished layout no drc or erc errors
Parts:
- removed TP39, TP44: TestPoint_Thimble, TestPoint:TestPoint_Loop_D3.50mm_Drill0.9mm_Beaded, symbol LiveAstra:TestPoint_Thimble
- added TP8: TestPoint_Thimble, LiveAstra:TestPoint_Loop_D3.50mm_Drill0.9mm_Beaded, symbol LiveAstra:TestPoint_Thimble
- C19, C20: footprint Capacitor_SMD:C_0402_1005Metric -> LiveAstra:C_0402_1005Metric
- R21: footprint Resistor_SMD:R_0805_2012Metric_Pad1.20x1.40mm_HandSolder -> LiveAstra:R_0805_2012Metric_Pad1.20x1.40mm_HandSolder
- R22: footprint Resistor_SMD:R_0402_1005Metric -> LiveAstra:R_0402_1005Metric
- TP24: renamed from TP36; footprint TestPoint:TestPoint_Loop_D3.50mm_Drill0.9mm_Beaded -> LiveAstra:TestPoint_Loop_D3.50mm_Drill0.9mm_Beaded; now not fitted; now left out of the parts list
- TP25: renamed from TP37; footprint TestPoint:TestPoint_Loop_D3.50mm_Drill0.9mm_Beaded -> LiveAstra:TestPoint_Loop_D3.50mm_Drill0.9mm_Beaded; now not fitted; now left out of the parts list
- TP26: renamed from TP38; footprint TestPoint:TestPoint_Loop_D3.50mm_Drill0.9mm_Beaded -> LiveAstra:TestPoint_Loop_D3.50mm_Drill0.9mm_Beaded; now not fitted; now left out of the parts list
- TP28: renamed from TP40; footprint TestPoint:TestPoint_Loop_D3.50mm_Drill0.9mm_Beaded -> LiveAstra:TestPoint_Loop_D3.50mm_Drill0.9mm_Beaded; now not fitted; now left out of the parts list
- TP29: renamed from TP41; footprint TestPoint:TestPoint_Loop_D3.50mm_Drill0.9mm_Beaded -> LiveAstra:TestPoint_Loop_D3.50mm_Drill0.9mm_Beaded; now not fitted; now left out of the parts list
- TP30: renamed from TP42; footprint TestPoint:TestPoint_Loop_D3.50mm_Drill0.9mm_Beaded -> LiveAstra:TestPoint_Loop_D3.50mm_Drill0.9mm_Beaded; now not fitted; now left out of the parts list
- TP31: renamed from TP43; footprint TestPoint:TestPoint_Loop_D3.50mm_Drill0.9mm_Beaded -> LiveAstra:TestPoint_Loop_D3.50mm_Drill0.9mm_Beaded; now not fitted; now left out of the parts list
- TP33: renamed from TP45; footprint TestPoint:TestPoint_Loop_D3.50mm_Drill0.9mm_Beaded -> LiveAstra:TestPoint_Loop_D3.50mm_Drill0.9mm_Beaded; now not fitted; now left out of the parts list
- TP34: renamed from TP46; footprint TestPoint:TestPoint_Loop_D3.50mm_Drill0.9mm_Beaded -> LiveAstra:TestPoint_Loop_D3.50mm_Drill0.9mm_Beaded; now not fitted; now left out of the parts list
- TP35: renamed from TP47; footprint TestPoint:TestPoint_Loop_D3.50mm_Drill0.9mm_Beaded -> LiveAstra:TestPoint_Loop_D3.50mm_Drill0.9mm_Beaded; now not fitted; now left out of the parts list
Connections:
- net +3V3: now also TP8.1
- net OE renamed LEVEL_SHIFTER_IO_OE

Commit message: workflow
Parts:
- TP24, TP25, TP26, TP28, TP29, TP30, TP31, TP33, TP34, TP35, TP8: now fitted
Changed lines of the file:
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@@
 		(in_bom no)
 		(on_board yes)
-		(dnp yes)
+		(dnp no)
 		(fields_autoplaced yes)
 		(property "Reference" "TP28"
@@
 			)
 		)
+		(property "Extra Value" ""
+			(at 129.54 91.44 0)
+			(effects
+				(font
+					(size 1.27 1.27)
+				)
+				(hide yes)
+			)
+		)
 		(pin "1"
 		)
@@
 			)
 		)
+		(property "Extra Value" ""
+			(at 106.68 83.82 0)
+			(effects
+				(font
+					(size 1.27 1.27)
+				)
+				(hide yes)
+			)
+		)
 		(pin "1"
 		)
@@
 		(in_bom no)
 		(on_board yes)
-		(dnp yes)
+		(dnp no)
 		(fields_autoplaced yes)
 		(property "Reference" "TP29"
@@
 			)
 		)
+		(property "Extra Value" ""
+			(at 129.54 106.68 0)
+			(effects
+				(font
+					(size 1.27 1.27)
+				)
+				(hide yes)
+			)
+		)
 		(pin "1"
 		)
@@
 		(in_bom no)
 		(on_board yes)
-		(dnp yes)
+		(dnp no)
 		(fields_autoplaced yes)
 		(property "Reference" "TP25"
@@
 			)
 		)
+		(property "Extra Value" ""
+			(at 81.28 116.84 0)
+			(effects
+				(font
+					(size 1.27 1.27)
+				)
+				(hide yes)
+			)
+		)
 		(pin "1"
 		)
@@
 			)
 		)
+		(property "Extra Value" ""
+			(at 152.4 88.9 0)
+			(effects
+				(font
+					(size 1.27 1.27)
+				)
+				(hide yes)
+			)
+		)
 		(pin "5"
 		)
@@
 		(in_bom no)
 		(on_board yes)
-		(dnp yes)
+		(dnp no)
 		(fields_autoplaced yes)
 		(property "Reference" "TP34"
@@
 			)
 		)
+		(property "Extra Value" ""
+			(at 215.9 116.84 0)
+			(effects
+				(font
+					(size 1.27 1.27)
+				)
+				(hide yes)
+			)
+		)
 		(pin "1"
 		)
@@
 		(in_bom no)
 		(on_board yes)
-		(dnp yes)
+		(dnp no)
 		(fields_autoplaced yes)
 		(property "Reference" "TP26"
@@
 			)
 		)
+		(property "Extra Value" ""
+			(at 106.68 111.76 0)
+			(effects
+				(font
+					(size 1.27 1.27)
+				)
+				(hide yes)
+			)
+		)
 		(pin "1"
 		)
@@
 			)
 		)
+		(property "Extra Value" ""
+			(at 88.9 76.2 0)
+			(effects
+				(font
+					(size 1.27 1.27)
+				)
+				(hide yes)
+			)
+		)
 		(pin "1"
 		)
@@
 		(in_bom no)
 		(on_board yes)
-		(dnp yes)
+		(dnp no)
 		(fields_autoplaced yes)
 		(property "Reference" "TP30"
@@
 			)
 		)
+		(property "Extra Value" ""
+			(at 167.64 106.68 0)
+			(effects
+				(font
+					(size 1.27 1.27)
+				)
+				(hide yes)
+			)
+		)
 		(pin "1"
 		)
@@
 		(in_bom no)
 		(on_board yes)
-		(dnp yes)
+		(dnp no)
 		(fields_autoplaced yes)
 		(property "Reference" "TP24"
@@
 			)
 		)
+		(property "Extra Value" ""
+			(at 55.88 121.92 0)
+			(effects
+				(font
+					(size 1.27 1.27)
+				)
+				(hide yes)
+			)
+		)
 		(pin "1"
 		)
@@
 		(in_bom no)
 		(on_board yes)
-		(dnp yes)
+		(dnp no)
 		(fields_autoplaced yes)
 		(property "Reference" "TP35"
@@
 			)
 		)
+		(property "Extra Value" ""
+			(at 243.84 121.92 0)
+			(effects
+				(font
+					(size 1.27 1.27)
+				)
+				(hide yes)
+			)
+		)
 		(pin "1"
 		)
@@
 		(in_bom no)
 		(on_board yes)
-		(dnp yes)
+		(dnp no)
 		(fields_autoplaced yes)
 		(property "Reference" "TP8"
@@
 			)
 		)
+		(property "Extra Value" ""
+			(at 127 48.26 0)
+			(effects
+				(font
+					(size 1.27 1.27)
+				)
+				(hide yes)
+			)
+		)
 		(pin "1"
 		)
@@
 		(in_bom no)
 		(on_board yes)
-		(dnp yes)
+		(dnp no)
 		(fields_autoplaced yes)
 		(property "Reference" "TP31"
@@
 			)
 		)
+		(property "Extra Value" ""
+			(at 177.8 48.26 0)
+			(effects
+				(font
+					(size 1.27 1.27)
+				)
+				(hide yes)
+			)
+		)
 		(pin "1"
 		)
@@
 			)
 		)
+		(property "Extra Value" ""
+			(at 114.3 58.42 0)
+			(effects
+				(font
+					(size 1.27 1.27)
+				)
+				(hide yes)
+			)
+		)
 		(pin "2"
 		)
@@
 			)
 		)
+		(property "Extra Value" ""
+			(at 190.5 58.42 0)
+			(effects
+				(font
+					(size 1.27 1.27)
+				)
+				(hide yes)
+			)
+		)
 		(pin "2"
 		)
@@
 		(in_bom no)
 		(on_board yes)
-		(dnp yes)
+		(dnp no)
 		(fields_autoplaced yes)
 		(property "Reference" "TP33"
@@
 			)
 		)
+		(property "Extra Value" ""
+			(at 190.5 111.76 0)
+			(effects
+				(font
+					(size 1.27 1.27)
+				)
+				(hide yes)
+			)
+		)

Commit message: workflow
Other:
- title: (none) -> 3V3 to 5V Logic Shifter
Changed lines of the file:
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@@
 	(generator_version "8.0")
 	(paper "A4")
+	(title_block
+		(title "3V3 to 5V Logic Shifter")
+	)
 	(junction
 		(at 190.5 114.3)
