File: 5V_Protection.kicad_sch (KiCad schematic)
At the start: 9 parts, among them U2 NCP361SNT1G

Commit message: Updated library name, updated and verified all footprints
Parts:
- C7, C8: symbol EASYEDA2KICAD:C_1uF_X5R_0402 -> LiveAstra:C_1uF_X5R_0402
- D1: symbol EASYEDA2KICAD:D_Schottky_1A_40V -> LiveAstra:D_Schottky_1A_40V
- LED2: symbol EASYEDA2KICAD:LED_RED_20mA_0603 -> LiveAstra:LED_RED_20mA_0603
- R8: symbol EASYEDA2KICAD:R_220Ohm_0402_62mW -> LiveAstra:R_220Ohm_0402_62mW
- TP6, TP8, TP9: symbol EASYEDA2KICAD:TestPoint_Thimble -> LiveAstra:TestPoint_Thimble
- U2: footprint EASYEDA2KICAD:TSOP-5_L3.0-W1.5-P0.95-BL -> LiveAstra:5V_PROTECTION_NCP361SNT1G_TSOP-5; symbol EASYEDA2KICAD:U_NCP361SNT1G_5V_Protection_IC_TSOP -> LiveAstra:U_NCP361SNT1G_5V_Protection_IC_TSOP
Changed lines of the file:
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@@
 	)
 	(symbol
-		(lib_id "EASYEDA2KICAD:C_1uF_X5R_0402")
+		(lib_id "LiveAstra:C_1uF_X5R_0402")
 		(at 127 91.44 90)
 		(unit 1)
@@
 	)
 	(symbol
-		(lib_id "EASYEDA2KICAD:LED_RED_20mA_0603")
+		(lib_id "LiveAstra:LED_RED_20mA_0603")
 		(at 208.28 99.06 0)
 		(unit 1)
@@
 	)
 	(symbol
-		(lib_id "EASYEDA2KICAD:D_Schottky_1A_40V")
+		(lib_id "LiveAstra:D_Schottky_1A_40V")
 		(at 86.36 101.6 180)
 		(unit 1)
@@
 	)
 	(symbol
-		(lib_id "EASYEDA2KICAD:TestPoint_Thimble")
+		(lib_id "LiveAstra:TestPoint_Thimble")
 		(at 177.8 124.46 0)
 		(unit 1)
@@
 	)
 	(symbol
-		(lib_id "EASYEDA2KICAD:TestPoint_Thimble")
+		(lib_id "LiveAstra:TestPoint_Thimble")
 		(at 185.42 81.28 0)
 		(unit 1)
@@
 	)
 	(symbol
-		(lib_id "EASYEDA2KICAD:R_220Ohm_0402_62mW")
+		(lib_id "LiveAstra:R_220Ohm_0402_62mW")
 		(at 241.3 99.06 180)
 		(unit 1)
@@
 	)
 	(symbol
-		(lib_id "EASYEDA2KICAD:U_NCP361SNT1G_5V_Protection_IC_TSOP")
+		(lib_id "LiveAstra:U_NCP361SNT1G_5V_Protection_IC_TSOP")
 		(at 152.4 101.6 0)
 		(unit 1)
@@
 			)
 		)
-		(property "Footprint" "EASYEDA2KICAD:TSOP-5_L3.0-W1.5-P0.95-BL"
+		(property "Footprint" "LiveAstra:5V_PROTECTION_NCP361SNT1G_TSOP-5"
 			(at 152.4 142.24 0)
 			(effects
@@
 	)
 	(symbol
-		(lib_id "EASYEDA2KICAD:C_1uF_X5R_0402")
+		(lib_id "LiveAstra:C_1uF_X5R_0402")
 		(at 170.18 91.44 270)
 		(unit 1)
@@
 	)
 	(symbol
-		(lib_id "EASYEDA2KICAD:TestPoint_Thimble")
+		(lib_id "LiveAstra:TestPoint_Thimble")
 		(at 114.3 81.28 0)
 		(unit 1)

Commit message: Finished layout no drc or erc errors
Parts:
- removed D1: SS14 Schottky, Diode_SMD:D_SMA, symbol LiveAstra:D_Schottky_1A_40V
- removed TP9: TestPoint_Thimble, TestPoint:TestPoint_Loop_D3.50mm_Drill0.9mm_Beaded, symbol LiveAstra:TestPoint_Thimble
- added D1: SS14 Schottky, LiveAstra:D_SMA_SS14_C2480, symbol LiveAstra:D_Schottky_SS14_1A_40V
- C7, C8: footprint Capacitor_SMD:C_0402_1005Metric -> LiveAstra:C_0402_1005Metric
- LED2: footprint LED_SMD:LED_0603_1608Metric -> LiveAstra:LED_0603_1608Metric
- R8: footprint Resistor_SMD:R_0402_1005Metric -> LiveAstra:R_0402_1005Metric
- TP6: footprint TestPoint:TestPoint_Loop_D3.50mm_Drill0.9mm_Beaded -> LiveAstra:TestPoint_Loop_D3.50mm_Drill0.9mm_Beaded; now not fitted; now left out of the parts list
- TP7: renamed from TP8; footprint TestPoint:TestPoint_Loop_D3.50mm_Drill0.9mm_Beaded -> LiveAstra:TestPoint_Loop_D3.50mm_Drill0.9mm_Beaded; now not fitted; now left out of the parts list
Connections:
- net 5V_IN: now also D1.1 (K)
- net VBUS: now also D1.2 (A)
Changed lines of the file:
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@@
 	(paper "A4")
-	(junction
-		(at 185.42 83.82)
-		(diameter 0)
-		(color 0 0 0 0)
-	)
 	(junction
 		(at 99.06 83.82)
@@
 	(wire
 		(pts
-			(xy 185.42 83.82) (xy 200.66 83.82)
+			(xy 170.18 83.82) (xy 200.66 83.82)
 		)
 		(stroke
@@
 	(wire
 		(pts
-			(xy 170.18 83.82) (xy 185.42 83.82)
-		)
-		(stroke
-			(width 0)
-			(type default)
-		)
-	)
-	(wire
-		(pts
 			(xy 127 83.82) (xy 144.78 83.82)
 		)
@@
 		(pts
 			(xy 99.06 83.82) (xy 114.3 83.82)
-		)
-		(stroke
-			(width 0)
-			(type default)
-		)
-	)
-	(wire
-		(pts
-			(xy 185.42 81.28) (xy 185.42 83.82)
 		)
 		(stroke
@@
 			)
 		)
-		(property "Footprint" "Capacitor_SMD:C_0402_1005Metric"
+		(property "Footprint" "LiveAstra:C_0402_1005Metric"
 			(at 139.7 91.44 0)
 			(effects
@@
 				(path "/9a751838-dce8-4d69-8a02-736625ac74e7/0db21d8e-3390-4d67-877f-0e5d98e37848/e21714b4-6921-40f8-8882-480f43314016"
 					(reference "C7")
+					(unit 1)
+				)
+			)
+		)
+	)
+	(symbol
+		(lib_id "LiveAstra:D_Schottky_SS14_1A_40V")
+		(at 86.36 101.6 180)
+		(unit 1)
+		(exclude_from_sim no)
+		(in_bom yes)
+		(on_board yes)
+		(dnp no)
+		(fields_autoplaced yes)
+		(property "Reference" "D1"
+			(at 86.74 92.71 0)
+			(effects
+				(font
+					(size 1.27 1.27)
+				)
+			)
+		)
+		(property "Value" "SS14 Schottky"
+			(at 86.74 95.25 0)
+			(effects
+				(font
+					(size 1.27 1.27)
+					(bold yes)
+				)
+			)
+		)
+		(property "Footprint" "LiveAstra:D_SMA_SS14_C2480"
+			(at 86.36 92.71 0)
+			(effects
+				(font
+					(size 1.27 1.27)
+				)
+				(hide yes)
+			)
+		)
+		(property "Datasheet" "https://lcsc.com/product-detail/Schottky-Barrier-Diodes-SBD_SS14_C2480.html"
+			(at 86.36 88.9 0)
+			(effects
+				(font
+					(size 1.27 1.27)
+				)
+				(hide yes)
+			)
+		)
+		(property "Description" "Schottky Barrier Diode"
+			(at 86.36 96.52 0)
+			(effects
+				(font
+					(size 1.27 1.27)
+				)
+				(hide yes)
+			)
+		)
+		(property "LCSC Part" "C2480"
+			(at 86.36 85.09 0)
+			(effects
+				(font
+					(size 1.27 1.27)
+				)
+				(hide yes)
+			)
+		)
+		(property "Extra Values" "40V Single 1A 550mV@1A"
+			(at 86.74 97.79 0)
+			(effects
+				(font
+					(size 0.762 0.762)
+					(bold yes)
+				)
+			)
+		)
+		(pin "1"
+		)
+		(pin "2"
+		)
+		(instances
+			(project "AstraControl"
+				(path "/9a751838-dce8-4d69-8a02-736625ac74e7/0db21d8e-3390-4d67-877f-0e5d98e37848/e21714b4-6921-40f8-8882-480f43314016"
+					(reference "D1")
 					(unit 1)
 				)
@@
 			)
 		)
-		(property "Footprint" "LED_SMD:LED_0603_1608Metric"
+		(property "Footprint" "LiveAstra:LED_0603_1608Metric"
 			(at 208.28 111.76 0)
 			(effects
@@
 	)
 	(symbol
-		(lib_id "LiveAstra:D_Schottky_1A_40V")
-		(at 86.36 101.6 180)
-		(unit 1)
-		(exclude_from_sim no)
-		(in_bom yes)
-		(on_board yes)
-		(dnp no)
-		(fields_autoplaced yes)
-		(property "Reference" "D1"
-			(at 86.74 92.71 0)
-			(effects
-				(font
-					(size 1.27 1.27)
-				)
-			)
-		)
-		(property "Value" "SS14 Schottky"
-			(at 86.74 95.25 0)
-			(effects
-				(font
-					(size 1.27 1.27)
-					(bold yes)
-				)
-			)
-		)
-		(property "Footprint" "Diode_SMD:D_SMA"
-			(at 86.36 92.71 0)
-			(effects
-				(font
-					(size 1.27 1.27)
-				)
-				(hide yes)
-			)
-		)
-		(property "Datasheet" "https://lcsc.com/product-detail/Schottky-Barrier-Diodes-SBD_SS14_C2480.html"
-			(at 86.36 88.9 0)
-			(effects
-				(font
-					(size 1.27 1.27)
-				)
-				(hide yes)
-			)
-		)
-		(property "Description" "Schottky Barrier Diode"
-			(at 86.36 96.52 0)
-			(effects
-				(font
-					(size 1.27 1.27)
-				)
-				(hide yes)
-			)
-		)
-		(property "LCSC Part" "C2480"
-			(at 86.36 85.09 0)
-			(effects
-				(font
-					(size 1.27 1.27)
-				)
-				(hide yes)
-			)
-		)
-		(property "Extra Values" "40V Single 1A 550mV@1A"
-			(at 86.74 97.79 0)
-			(effects
-				(font
-					(size 0.762 0.762)
-					(bold yes)
-				)
-			)
-		)
-		(pin "2"
-		)
-		(pin "1"
-		)
-		(instances
-			(project "AstraControl"
-				(path "/9a751838-dce8-4d69-8a02-736625ac74e7/0db21d8e-3390-4d67-877f-0e5d98e37848/e21714b4-6921-40f8-8882-480f43314016"
-					(reference "D1")
-					(unit 1)
-				)
-			)
-		)
-	)
-	(symbol
 		(lib_id "LiveAstra:TestPoint_Thimble")
 		(at 177.8 124.46 0)
 		(unit 1)
 		(exclude_from_sim no)
-		(in_bom yes)
+		(in_bom no)
 		(on_board yes)
-		(dnp no)
+		(dnp yes)
 		(fields_autoplaced yes)
-		(property "Reference" "TP8"
+		(property "Reference" "TP7"
 			(at 180.34 118.6476 0)
 			(effects
@@
 			)
 		)
-		(property "Footprint" "TestPoint:TestPoint_Loop_D3.50mm_Drill0.9mm_Beaded"
+		(property "Footprint" "LiveAstra:TestPoint_Loop_D3.50mm_Drill0.9mm_Beaded"
 			(at 177.8 139.7 0)
 			(effects
@@
 			(project "AstraControl"
 				(path "/9a751838-dce8-4d69-8a02-736625ac74e7/0db21d8e-3390-4d67-877f-0e5d98e37848/e21714b4-6921-40f8-8882-480f43314016"
-					(reference "TP8")
+					(reference "TP7")
 					(unit 1)
 				)
@@
 	)
 	(symbol
-		(lib_id "LiveAstra:TestPoint_Thimble")
-		(at 185.42 81.28 0)
-		(unit 1)
-		(exclude_from_sim no)
-		(in_bom yes)
-		(on_board yes)
-		(dnp no)
-		(fields_autoplaced yes)
-		(property "Reference" "TP9"
-			(at 187.96 75.4676 0)
-			(effects
-				(font
-					(size 1.27 1.27)
-				)
-				(justify left)
-			)
-		)
-		(property "Value" "TestPoint_Thimble"
-			(at 185.42 91.44 0)
-			(effects
-				(font
-					(size 1.27 1.27)
-				)
-				(hide yes)
-			)
-		)
-		(property "Footprint" "TestPoint:TestPoint_Loop_D3.50mm_Drill0.9mm_Beaded"
-			(at 185.42 96.52 0)
-			(effects
-				(font
-					(size 1.27 1.27)
-				)
-				(hide yes)
-			)
-		)
-		(property "Datasheet" ""
-			(at 185.42 76.2 90)
-			(effects
-				(font
-					(size 1.27 1.27)
-				)
-				(hide yes)
-			)
-		)
-		(property "Description" ""
-			(at 185.42 76.2 90)
-			(effects
-				(font
-					(size 1.27 1.27)
-				)
-				(hide yes)
-			)
-		)
-		(property "LCSC Part" "C5277086"
-			(at 185.42 101.6 0)
-			(effects
-				(font
-					(size 1.27 1.27)
-				)
-				(hide yes)
-			)
-		)
-		(property "Extra Values" "Test Plug"
-			(at 187.96 78.0076 0)
-			(effects
-				(font
-					(size 0.762 0.762)
-					(bold yes)
-				)
-				(justify left)
-			)
-		)
-		(pin "1"
-		)
-		(instances
-			(project "AstraControl"
-				(path "/9a751838-dce8-4d69-8a02-736625ac74e7/0db21d8e-3390-4d67-877f-0e5d98e37848/e21714b4-6921-40f8-8882-480f43314016"
-					(reference "TP9")
-					(unit 1)
-				)
-			)
-		)
-	)
-	(symbol
 		(lib_id "power:GND")
 		(at 170.18 96.52 0)
@@
 			)
 		)
-		(property "Footprint" "Resistor_SMD:R_0402_1005Metric"
+		(property "Footprint" "LiveAstra:R_0402_1005Metric"
 			(at 241.3 90.17 0)
 			(effects
@@
 			)
 		)
-		(property "Footprint" "Capacitor_SMD:C_0402_1005Metric"
+		(property "Footprint" "LiveAstra:C_0402_1005Metric"
 			(at 157.48 91.44 0)
 			(effects
@@
 		(unit 1)
 		(exclude_from_sim no)
-		(in_bom yes)
+		(in_bom no)
 		(on_board yes)
-		(dnp no)
+		(dnp yes)
 		(fields_autoplaced yes)
 		(property "Reference" "TP6"
@@
 			)
 		)
-		(property "Footprint" "TestPoint:TestPoint_Loop_D3.50mm_Drill0.9mm_Beaded"
+		(property "Footprint" "LiveAstra:TestPoint_Loop_D3.50mm_Drill0.9mm_Beaded"
 			(at 114.3 96.52 0)
 			(effects

Commit message: Work on kibot
Changed lines of the file:
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@@
-		)
-	)
-	(polyline
-		(pts
-			(xy 135.5667 47.3) (xy 135.5667 47.3)
-		)
-		(stroke
-			(width -0.0001)
-			(type solid)
-		)
-	)
-	(polyline
-		(pts
-			(xy 135.5798 48.7555) (xy 135.5928 48.7565) (xy 135.6057 48.7581) (xy 135.6185 48.7603) (xy 135.6312 48.7632)
-			(xy 135.6436 48.7666) (xy 135.6559 48.7707) (xy 135.6679 48.7753) (xy 135.6797 48.7806) (xy 135.6913 48.7864)
-			(xy 135.7025 48.7927) (xy 135.7135 48.7997) (xy 135.7241 48.8071) (xy 135.7343 48.8151) (xy 135.7442 48.8237)
-			(xy 135.7538 48.8327) (xy 135.7628 48.8422) (xy 135.7713 48.8521) (xy 135.7793 48.8624) (xy 135.7868 48.873)
-			(xy 135.7937 48.8839) (xy 135.8001 48.8952) (xy 135.8059 48.9067) (xy 135.8111 48.9185) (xy 135.8158 48.9306)
-			(xy 135.8198 48.9428) (xy 135.8233 48.9553) (xy 135.8261 48.9679) (xy 135.8284 48.9807) (xy 135.83 48.9936)
-			(xy 135.8309 49.0067) (xy 135.8312 49.0198) (xy 135.8312 50.475) (xy 136.0958 50.475) (xy 136.0958 50.7396)
-			(xy 135.3021 50.7396) (xy 135.3021 50.475) (xy 135.5667 50.475) (xy 135.5667 49.0198) (xy 135.1698 49.0198)
-			(xy 135.1698 48.7552) (xy 135.5667 48.7552) (xy 135.5798 48.7555)
-		)
-		(stroke
-			(width -0.0001)
-			(type solid)
-		)
-		(fill
-			(type color)
-			(color 34 187 51 1)
-		)
-	)
-	(polyline
-		(pts
-			(xy 135.6716 47.3026) (xy 135.7759 47.3104) (xy 135.8792 47.3232) (xy 135.9815 47.341) (xy 136.0826 47.3638)
-			(xy 136.1823 47.3915) (xy 136.2804 47.4239) (xy 136.3767 47.4611) (xy 136.4711 47.5029) (xy 136.5634 47.5494)
-			(xy 136.6534 47.6003) (xy 136.741 47.6556) (xy 136.826 47.7153) (xy 136.9081 47.7793) (xy 136.9873 47.8476)
-			(xy 137.0634 47.92) (xy 137.1358 47.996) (xy 137.204 48.0752) (xy 137.268 48.1574) (xy 137.3277 48.2423)
-			(xy 137.3831 48.3299) (xy 137.434 48.4199) (xy 137.4804 48.5123) (xy 137.5222 48.6067) (xy 137.5594 48.703)
-			(xy 137.5918 48.8011) (xy 137.6195 48.9007) (xy 137.6423 49.0018) (xy 137.6601 49.1041) (xy 137.673 49.2075)
-			(xy 137.6807 49.3117) (xy 137.6833 49.4167) (xy 137.6818 49.4967) (xy 137.6773 49.5761) (xy 137.6699 49.6549)
-			(xy 137.6596 49.7331) (xy 137.6465 49.8104) (xy 137.6305 49.887) (xy 137.6118 49.9626) (xy 137.5904 50.0373)
-			(xy 137.5663 50.111) (xy 137.5396 50.1836) (xy 137.5103 50.255) (xy 137.4784 50.3252) (xy 137.4441 50.3942)
-			(xy 137.4073 50.4618) (xy 137.3682 50.5279) (xy 137.3266 50.5926) (xy 137.2827 50.6558) (xy 137.2366 50.7173)
-			(xy 137.1882 50.7771) (xy 137.1377 50.8352) (xy 137.085 50.8915) (xy 137.0302 50.9459) (xy 136.9734 50.9984)
-			(xy 136.9145 51.0488) (xy 136.8537 51.0972) (xy 136.791 51.1434) (xy 136.7264 51.1875) (xy 136.6599 51.2292)
-			(xy 136.5917 51.2687) (xy 136.5217 51.3057) (xy 136.45 51.3402) (xy 136.3767 51.3722) (xy 136.2271 51.4277)
-			(xy 136.0753 51.4714) (xy 135.922 51.5034) (xy 135.7677 51.5239) (xy 135.6131 51.5329) (xy 135.4589 51.5306)
-			(xy 135.3055 51.5172) (xy 135.1537 51.4927) (xy 135.0041 51.4572) (xy 134.8573 51.411) (xy 134.7139 51.354)
-			(xy 134.5745 51.2865) (xy 134.4398 51.2086) (xy 134.3104 51.1203) (xy 134.1869 51.0219) (xy 134.07 50.9134)
-			(xy 133.9614 50.7964) (xy 133.863 50.6729) (xy 133.7747 50.5435) (xy 133.6968 50.4088) (xy 133.6293 50.2694)
-			(xy 133.5724 50.126) (xy 133.5261 49.9792) (xy 133.4907 49.8296) (xy 133.4662 49.6778) (xy 133.4527 49.5245)
-			(xy 133.4517 49.4573) (xy 133.715 49.4573) (xy 133.7229 49.5926) (xy 133.7408 49.7276) (xy 133.7688 49.8617)
-			(xy 133.807 49.9945) (xy 133.8556 50.1254) (xy 133.9138 50.2523) (xy 133.9807 50.3733) (xy 134.0557 50.4879)
-			(xy 134.1385 50.596) (xy 134.2286 50.6973) (xy 134.3254 50.7913) (xy 134.4286 50.8779) (xy 134.5377 50.9566)
-			(xy 134.6522 51.0273) (xy 134.7717 51.0895) (xy 134.8956 51.143) (xy 135.0236 51.1874) (xy 135.1552 51.2225)
-			(xy 135.2898 51.248) (xy 135.4272 51.2635) (xy 135.5667 51.2687) (xy 135.6585 51.2665) (xy 135.7497 51.2597)
-			(xy 135.8402 51.2485) (xy 135.9297 51.2328) (xy 136.0181 51.2129) (xy 136.1053 51.1887) (xy 136.1911 51.1603)
-			(xy 136.2754 51.1278) (xy 136.358 51.0912) (xy 136.4388 51.0506) (xy 136.5176 51.006) (xy 136.5942 50.9576)
-			(xy 136.6685 50.9053) (xy 136.7404 50.8493) (xy 136.8097 50.7896) (xy 136.8763 50.7263) (xy 136.9396 50.6597)
-			(xy 136.9993 50.5904) (xy 137.0553 50.5185) (xy 137.1076 50.4442) (xy 137.156 50.3676) (xy 137.2006 50.2888)
-			(xy 137.2412 50.208) (xy 137.2778 50.1254) (xy 137.3103 50.0411) (xy 137.3387 49.9553) (xy 137.3629 49.8681)
-			(xy 137.3828 49.7797) (xy 137.3985 49.6902) (xy 137.4097 49.5997) (xy 137.4165 49.5085) (xy 137.4187 49.4167)
-			(xy 137.4174 49.3467) (xy 137.4135 49.2772) (xy 137.407 49.2082) (xy 137.398 49.1398) (xy 137.3865 49.0721)
-			(xy 137.3725 49.0052) (xy 137.3562 48.939) (xy 137.3374 48.8736) (xy 137.3163 48.8091) (xy 137.293 48.7456)
-			(xy 137.2673 48.6831) (xy 137.2395 48.6217) (xy 137.2094 48.5613) (xy 137.1773 48.5022) (xy 137.143 48.4443)
-			(xy 137.1066 48.3877) (xy 137.0682 48.3325) (xy 137.0279 48.2786) (xy 136.9855 48.2263) (xy 136.9413 48.1754)
-			(xy 136.8952 48.1262) (xy 136.8473 48.0786) (xy 136.7975 48.0327) (xy 136.746 47.9885) (xy 136.6928 47.9462)
-			(xy 136.6379 47.9057) (xy 136.5814 47.8672) (xy 136.5233 47.8307) (xy 136.4636 47.7962) (xy 136.4023 47.7638)
-			(xy 136.3396 47.7336) (xy 136.2754 47.7056) (xy 136.1445 47.657) (xy 136.0117 47.6188) (xy 135.8776 47.5908)
-			(xy 135.7426 47.5729) (xy 135.6073 47.565) (xy 135.4723 47.567) (xy 135.3382 47.5787) (xy 135.2053 47.6002)
-			(xy 135.0744 47.6312) (xy 134.946 47.6717) (xy 134.8205 47.7215) (xy 134.6986 47.7805) (xy 134.5807 47.8487)
-			(xy 134.4675 47.926) (xy 134.3594 48.0121) (xy 134.257 48.107) (xy 134.1621 48.2094) (xy 134.076 48.3175)
-			(xy 133.9987 48.4307) (xy 133.9305 48.5486) (xy 133.8715 48.6705) (xy 133.8217 48.796) (xy 133.7812 48.9244)
-			(xy 133.7502 49.0553) (xy 133.7287 49.1882) (xy 133.717 49.3223) (xy 133.715 49.4573) (xy 133.4517 49.4573)
-			(xy 133.4504 49.3702) (xy 133.4595 49.2156) (xy 133.4799 49.0614) (xy 133.5119 48.908) (xy 133.5556 48.7563)
-			(xy 133.6111 48.6067) (xy 133.6777 48.4616) (xy 133.7541 48.3234) (xy 133.8399 48.1924) (xy 133.9345 48.0688)
-			(xy 134.0374 47.9531) (xy 134.1481 47.8456) (xy 134.266 47.7467) (xy 134.3907 47.6567) (xy 134.5216 47.576)
-			(xy 134.6581 47.5049) (xy 134.7997 47.4437) (xy 134.946 47.3929) (xy 135.0964 47.3528) (xy 135.2503 47.3237)
-			(xy 135.4072 47.306) (xy 135.5667 47.3) (xy 135.6716 47.3026)
-		)
-		(stroke
-			(width -0.0001)
-			(type solid)
-		)
-		(fill
-			(type color)
-			(color 34 187 51 1)
-		)
-	)
-	(polyline
-		(pts
-			(xy 135.5803 47.9618) (xy 135.5937 47.9628) (xy 135.607 47.9645) (xy 135.62 47.9668) (xy 135.6328 47.9698)
-			(xy 135.6453 47.9734) (xy 135.6576 47.9775) (xy 135.6697 47.9823) (xy 135.6814 47.9875) (xy 135.6928 47.9934)
-			(xy 135.7039 47.9998) (xy 135.7146 48.0066) (xy 135.725 48.014) (xy 135.735 48.0219) (xy 135.7446 48.0302)
-			(xy 135.7538 48.039) (xy 135.7625 48.0481) (xy 135.7708 48.0577) (xy 135.7787 48.0677) (xy 135.7861 48.0781)
-			(xy 135.7929 48.0888) (xy 135.7993 48.0999) (xy 135.8052 48.1113) (xy 135.8105 48.1231) (xy 135.8152 48.1351)
-			(xy 135.8194 48.1474) (xy 135.8229 48.1599) (xy 135.8259 48.1727) (xy 135.8282 48.1857) (xy 135.8299 48.199)
-			(xy 135.8309 48.2124) (xy 135.8312 48.226) (xy 135.8309 48.2397) (xy 135.8299 48.2531) (xy 135.8282 48.2663)
-			(xy 135.8259 48.2794) (xy 135.8229 48.2922) (xy 135.8194 48.3047) (xy 135.8152 48.317) (xy 135.8105 48.329)
-			(xy 135.8052 48.3407) (xy 135.7993 48.3522) (xy 135.7929 48.3632) (xy 135.7861 48.374) (xy 135.7787 48.3843)
-			(xy 135.7708 48.3943) (xy 135.7625 48.4039) (xy 135.7538 48.4131) (xy 135.7446 48.4219) (xy 135.735 48.4302)
-			(xy 135.725 48.4381) (xy 135.7146 48.4454) (xy 135.7039 48.4523) (xy 135.6928 48.4587) (xy 135.6814 48.4645)
-			(xy 135.6697 48.4698) (xy 135.6576 48.4746) (xy 135.6453 48.4787) (xy 135.6328 48.4823) (xy 135.62 48.4852)
-			(xy 135.607 48.4876) (xy 135.5937 48.4893) (xy 135.5803 48.4903) (xy 135.5667 48.4906) (xy 135.5531 48.4903)
-			(xy 135.5396 48.4893) (xy 135.5264 48.4876) (xy 135.5133 48.4852) (xy 135.5005 48.4823) (xy 135.488 48.4787)
-			(xy 135.4757 48.4746) (xy 135.4637 48.4698) (xy 135.452 48.4645) (xy 135.4406 48.4587) (xy 135.4295 48.4523)
-			(xy 135.4187 48.4454) (xy 135.4084 48.4381) (xy 135.3984 48.4302) (xy 135.3888 48.4219) (xy 135.3796 48.4131)
-			(xy 135.3708 48.4039) (xy 135.3625 48.3943) (xy 135.3546 48.3843) (xy 135.3473 48.374) (xy 135.3404 48.3632)
-			(xy 135.334 48.3522) (xy 135.3282 48.3407) (xy 135.3229 48.329) (xy 135.3181 48.317) (xy 135.314 48.3047)
-			(xy 135.3104 48.2922) (xy 135.3075 48.2794) (xy 135.3051 48.2663) (xy 135.3034 48.2531) (xy 135.3024 48.2397)
-			(xy 135.3021 48.226) (xy 135.3024 48.2124) (xy 135.3034 48.199) (xy 135.3051 48.1857) (xy 135.3075 48.1727)
-			(xy 135.3104 48.1599) (xy 135.314 48.1474) (xy 135.3181 48.1351) (xy 135.3229 48.1231) (xy 135.3282 48.1113)
-			(xy 135.334 48.0999) (xy 135.3404 48.0888) (xy 135.3473 48.0781) (xy 135.3546 48.0677) (xy 135.3625 48.0577)
-			(xy 135.3708 48.0481) (xy 135.3796 48.039) (xy 135.3888 48.0302) (xy 135.3984 48.0219) (xy 135.4084 48.014)
-			(xy 135.4187 48.0066) (xy 135.4295 47.9998) (xy 135.4406 47.9934) (xy 135.452 47.9875) (xy 135.4637 47.9823)
-			(xy 135.4757 47.9775) (xy 135.488 47.9734) (xy 135.5005 47.9698) (xy 135.5133 47.9668) (xy 135.5264 47.9645)
-			(xy 135.5396 47.9628) (xy 135.5531 47.9618) (xy 135.5667 47.9615) (xy 135.5803 47.9618)
-		)
-		(stroke
-			(width -0.0001)
-			(type solid)
-		)
-		(fill
-			(type color)
-			(color 34 187 51 1)
 		)
 	)

Commit message: workflow
Parts:
- TP6, TP7: now fitted
Changed lines of the file:
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@@
+			)
+		)
+		(property "Extra Value" ""
+			(at 127 91.44 0)
+			(effects
+				(font
+					(size 1.27 1.27)
+				)
+				(hide yes)
 			)
 		)
@@
 			)
 		)
+		(property "Extra Value" ""
+			(at 86.36 101.6 0)
+			(effects
+				(font
+					(size 1.27 1.27)
+				)
+				(hide yes)
+			)
+		)
 		(pin "1"
 		)
@@
 			)
 		)
+		(property "Extra Value" ""
+			(at 208.28 99.06 0)
+			(effects
+				(font
+					(size 1.27 1.27)
+				)
+				(hide yes)
+			)
+		)
 		(pin "2"
 		)
@@
 		(in_bom no)
 		(on_board yes)
-		(dnp yes)
+		(dnp no)
 		(fields_autoplaced yes)
 		(property "Reference" "TP7"
@@
 			)
 		)
+		(property "Extra Value" ""
+			(at 177.8 124.46 0)
+			(effects
+				(font
+					(size 1.27 1.27)
+				)
+				(hide yes)
+			)
+		)
 		(pin "1"
 		)
@@
 			)
 		)
+		(property "Extra Value" ""
+			(at 241.3 99.06 0)
+			(effects
+				(font
+					(size 1.27 1.27)
+				)
+				(hide yes)
+			)
+		)
 		(pin "2"
 		)
@@
 			)
 		)
+		(property "Extra Value" ""
+			(at 152.4 101.6 0)
+			(effects
+				(font
+					(size 1.27 1.27)
+				)
+				(hide yes)
+			)
+		)
 		(pin "2"
 		)
@@
 			)
 		)
+		(property "Extra Value" ""
+			(at 170.18 91.44 0)
+			(effects
+				(font
+					(size 1.27 1.27)
+				)
+				(hide yes)
+			)
+		)
 		(pin "1"
 		)
@@
 		(in_bom no)
 		(on_board yes)
-		(dnp yes)
+		(dnp no)
 		(fields_autoplaced yes)
 		(property "Reference" "TP6"
@@
 			)
 		)
+		(property "Extra Value" ""
+			(at 114.3 81.28 0)
+			(effects
+				(font
+					(size 1.27 1.27)
+				)
+				(hide yes)
+			)
+		)

Commit message: workflow
Other:
- title: (none) -> 5V Protection
Changed lines of the file:
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@@
 	(generator_version "8.0")
 	(paper "A4")
+	(title_block
+		(title "5V Protection")
+	)
 	(junction
 		(at 99.06 83.82)
