File: 5v_gpio_connectors.kicad_sch (KiCad schematic)
At the start: 2 parts, among them CN2 4P JST VH, CN3 4P JST VH

Commit message: Updated library name, updated and verified all footprints
Parts:
- CN2, CN3: footprint EASYEDA2KICAD:JST_VH_B4P-VH-B_1x04_P3.96mm_Vertical -> LiveAstra:JST_VH_B4P-VH-B_1x04_P3.96mm_Vertical; symbol EASYEDA2KICAD:JST_VH_4PIN_10A_250V -> LiveAstra:JST_VH_4PIN_10A_250V
Changed lines of the file:
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@@
 	)
 	(symbol
-		(lib_id "EASYEDA2KICAD:+5V_IN")
+		(lib_id "LiveAstra:+5V_IN")
 		(at 127 114.3 0)
 		(unit 1)
@@
 	)
 	(symbol
-		(lib_id "EASYEDA2KICAD:+5V_IN")
+		(lib_id "LiveAstra:+5V_IN")
 		(at 127 78.74 0)
 		(unit 1)
@@
 	)
 	(symbol
-		(lib_id "EASYEDA2KICAD:JST_VH_4PIN_10A_250V")
+		(lib_id "LiveAstra:JST_VH_4PIN_10A_250V")
 		(at 157.48 83.82 0)
 		(unit 1)
@@
 			)
 		)
-		(property "Footprint" "EASYEDA2KICAD:JST_VH_B4P-VH-B_1x04_P3.96mm_Vertical"
+		(property "Footprint" "LiveAstra:JST_VH_B4P-VH-B_1x04_P3.96mm_Vertical"
 			(at 157.48 104.14 0)
 			(effects
@@
 	)
 	(symbol
-		(lib_id "EASYEDA2KICAD:JST_VH_4PIN_10A_250V")
+		(lib_id "LiveAstra:JST_VH_4PIN_10A_250V")
 		(at 157.48 119.38 0)
 		(unit 1)
@@
 			)
 		)
-		(property "Footprint" "EASYEDA2KICAD:JST_VH_B4P-VH-B_1x04_P3.96mm_Vertical"
+		(property "Footprint" "LiveAstra:JST_VH_B4P-VH-B_1x04_P3.96mm_Vertical"
 			(at 157.48 139.7 0)
 			(effects

Commit message: workflow
Other:
- title: (none) -> 5V GPIO Connectors
Changed lines of the file:
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@@
 	(generator_version "8.0")
 	(paper "A4")
+	(title_block
+		(title "5V GPIO Connectors")
+	)
 	(wire
 		(pts
