File: AstraControl.kicad_sch (KiCad schematic)
At the start: 0 parts

Commit message: workflow
Other:
- note added: "In review"
- note removed: "Draft"
- title: Astra Beam High Power RGBW LED Controller -> AstraControl - ESP32 Based Controller
Changed lines of the file:
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@@
 	(paper "A4")
 	(title_block
-		(title "Astra Beam High Power RGBW LED Controller")
+		(title "AstraControl - ESP32 Based Controller")
 		(rev "A")
 		(company "LiveAstra Technologies")
@@
 		)
 	)
-	(text "Draft"
+	(text "In review"
 		(exclude_from_sim no)
 		(at 35 52.5 0)
