File: button_status_uart_i2s.kicad_sch (KiCad schematic)
At the start: 16 parts, among them CN10 JST_ZH_6PIN_1A_250V, CN8 4P JST ZH, CN9 4P JST ZH

Commit message: Ready for kibot
Connections:
- net GPIO_12_BUTTON renamed BUTTON
- net GPIO_12_BUTTON_0 renamed BUTTON_0
- net GPIO_12_BUTTON_CONN renamed BUTTON_CONN
- net GPIO_13_STATUS_LED renamed STATUS_LED
- net GPIO_13_STATUS_LED_CONN renamed STATUS_LED_CONN
- net GPIO_14_I2S_WS renamed I2S_WS
- net GPIO_21_I2S_SCK renamed I2S_SCK
- net GPIO_47_I2S_SD renamed I2S_SD
- net GPIO_48_I2S_LR renamed I2S_LR
Other:
- moved on the sheet: R33
Changed lines of the file:
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@@
 	(wire
 		(pts
-			(xy 76.2 109.22) (xy 109.22 109.22)
+			(xy 76.2 109.22) (xy 96.52 109.22)
 		)
 		(stroke
@@
 	(wire
 		(pts
-			(xy 119.38 109.22) (xy 127 109.22)
+			(xy 106.68 109.22) (xy 127 109.22)
 		)
 		(stroke
@@
 		)
 	)
-	(label "GPIO_12_BUTTON_CONN"
+	(label "BUTTON_CONN"
 		(at 129.54 71.12 0)
 		(fields_autoplaced yes)
@@
 		)
 	)
-	(label "GPIO_13_STATUS_LED_CONN"
+	(label "STATUS_LED_CONN"
 		(at 129.54 109.22 0)
 		(fields_autoplaced yes)
@@
 		)
 	)
-	(label "GPIO_12_BUTTON_0"
+	(label "BUTTON_0"
 		(at 91.44 71.12 0)
 		(fields_autoplaced yes)
@@
 		)
 	)
+	(hierarchical_label "I2S_SCK"
+		(shape input)
+		(at 76.2 152.4 180)
+		(fields_autoplaced yes)
+		(effects
+			(font
+				(size 1.27 1.27)
+			)
+			(justify right)
+		)
+	)
 	(hierarchical_label "UART_RX"
 		(shape output)
@@
 		)
 	)
-	(hierarchical_label "GPIO_12_BUTTON"
+	(hierarchical_label "I2S_WS"
 		(shape input)
-		(at 76.2 71.12 180)
+		(at 76.2 167.64 180)
 		(fields_autoplaced yes)
 		(effects
@@
 		)
 	)
-	(hierarchical_label "GPIO_48_I2S_LR"
-		(shape input)
-		(at 76.2 182.88 180)
+	(hierarchical_label "I2S_SD"
+		(shape bidirectional)
+		(at 76.2 134.62 180)
 		(fields_autoplaced yes)
 		(effects
@@
 		)
 	)
+	(hierarchical_label "I2S_LR"
+		(shape input)
+		(at 76.2 182.88 180)
+		(fields_autoplaced yes)
+		(effects
+			(font
+				(size 1.27 1.27)
+			)
+			(justify right)
+		)
+	)
+	(hierarchical_label "STATUS_LED"
+		(shape input)
+		(at 76.2 109.22 180)
+		(fields_autoplaced yes)
+		(effects
+			(font
+				(size 1.27 1.27)
+			)
+			(justify right)
+		)
+	)
 	(hierarchical_label "UART_TX"
 		(shape input)
@@
 		)
 	)
-	(hierarchical_label "GPIO_14_I2S_WS"
+	(hierarchical_label "BUTTON"
 		(shape input)
-		(at 76.2 167.64 180)
-		(fields_autoplaced yes)
-		(effects
-			(font
-				(size 1.27 1.27)
-			)
-			(justify right)
-		)
-	)
-	(hierarchical_label "GPIO_13_STATUS_LED"
-		(shape input)
-		(at 76.2 109.22 180)
-		(fields_autoplaced yes)
-		(effects
-			(font
-				(size 1.27 1.27)
-			)
-			(justify right)
-		)
-	)
-	(hierarchical_label "GPIO_47_I2S_SD"
-		(shape output)
-		(at 76.2 134.62 180)
-		(fields_autoplaced yes)
-		(effects
-			(font
-				(size 1.27 1.27)
-			)
-			(justify right)
-		)
-	)
-	(hierarchical_label "GPIO_21_I2S_SCK"
-		(shape input)
-		(at 76.2 152.4 180)
+		(at 76.2 71.12 180)
 		(fields_autoplaced yes)
 		(effects
@@
 	(symbol
 		(lib_id "LiveAstra:R_0Ohm_0805_125mW")
-		(at 114.3 109.22 0)
+		(at 101.6 109.22 0)
 		(unit 1)
 		(exclude_from_sim no)
@@
 		(dnp no)
 		(property "Reference" "R33"
-			(at 114.3 101.6 0)
+			(at 101.6 101.6 0)
 			(effects
 				(font
@@
 		)
 		(property "Value" "0"
-			(at 114.3 104.14 0)
+			(at 101.6 104.14 0)
 			(effects
 				(font
@@
 		)
 		(property "Footprint" "LiveAstra:R_0805_2012Metric_Pad1.20x1.40mm_HandSolder"
-			(at 114.3 121.92 0)
+			(at 101.6 121.92 0)
 			(effects
 				(font
@@
 		)
 		(property "Datasheet" "https://lcsc.com/product-detail/Chip-Resistor-Surface-Mount-UniOhm_0R-0R0-1_C17477.html"
-			(at 114.3 118.11 0)
+			(at 101.6 118.11 0)
 			(effects
 				(font
@@
 		)
 		(property "Description" "Thick Film Resistors"
-			(at 114.3 114.3 0)
+			(at 101.6 114.3 0)
 			(effects
 				(font
@@
 		)
 		(property "LCSC Part" "C17477"
-			(at 114.3 125.73 0)
+			(at 101.6 125.73 0)
 			(effects
 				(font
@@
 		)
 		(property "Extra Values" "150V ±1% 0805"
-			(at 114.3 106.68 0)
-			(effects
-				(font
+			(at 101.6 106.68 0)
+			(effects
+				(font

Commit message: Work on kibot
Parts:
- CN10: Extra Values 6PIN 1A 1.5mm -> 6PIN 1A 1.5mm
- CN8, CN9: Extra Values 4PIN 1A 1.5mm -> 4PIN 1A 1.5mm
Changed lines of the file:
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@@
 			)
 		)
-		(property "Extra Values" "4PIN 1A 1.5mm "
+		(property "Extra Values" "4PIN 1A 1.5mm"
 			(at 179.07 40.6399 0)
 			(effects
@@
 			)
 		)
-		(property "Extra Values" "4PIN 1A 1.5mm "
+		(property "Extra Values" "4PIN 1A 1.5mm"
 			(at 179.07 71.1199 0)
 			(effects
@@
 			)
 		)
-		(property "Extra Values" "6PIN 1A 1.5mm "
+		(property "Extra Values" "6PIN 1A 1.5mm"
 			(at 179.07 138.4299 0)
 			(effects

Commit message: workflow
Changed lines of the file:
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@@
 	)
 	(hierarchical_label "I2S_SD"
-		(shape bidirectional)
+		(shape output)
 		(at 76.2 134.62 180)
 		(fields_autoplaced yes)

Commit message: workflow
Parts:
- TP48, TP49, TP50, TP51, TP52, TP53, TP54, TP55: now fitted
Changed lines of the file:
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@@
 		(in_bom no)
 		(on_board yes)
-		(dnp yes)
+		(dnp no)
 		(fields_autoplaced yes)
 		(property "Reference" "TP51"
@@
 			)
 		)
+		(property "Extra Value" ""
+			(at 127 132.08 0)
+			(effects
+				(font
+					(size 1.27 1.27)
+				)
+				(hide yes)
+			)
+		)
 		(pin "1"
 		)
@@
 			)
 		)
+		(property "Extra Value" ""
+			(at 172.72 38.1 0)
+			(effects
+				(font
+					(size 1.27 1.27)
+				)
+				(hide yes)
+			)
+		)
 		(pin "1"
 		)
@@
 		(in_bom no)
 		(on_board yes)
-		(dnp yes)
+		(dnp no)
 		(fields_autoplaced yes)
 		(property "Reference" "TP49"
@@
 			)
 		)
+		(property "Extra Value" ""
+			(at 127 68.58 0)
+			(effects
+				(font
+					(size 1.27 1.27)
+				)
+				(hide yes)
+			)
+		)
 		(pin "1"
 		)
@@
 		(in_bom no)
 		(on_board yes)
-		(dnp yes)
+		(dnp no)
 		(fields_autoplaced yes)
 		(property "Reference" "TP50"
@@
 			)
 		)
+		(property "Extra Value" ""
+			(at 127 106.68 0)
+			(effects
+				(font
+					(size 1.27 1.27)
+				)
+				(hide yes)
+			)
+		)
 		(pin "1"
 		)
@@
 		(in_bom no)
 		(on_board yes)
-		(dnp yes)
+		(dnp no)
 		(fields_autoplaced yes)
 		(property "Reference" "TP54"
@@
 			)
 		)
+		(property "Extra Value" ""
+			(at 127 180.34 0)
+			(effects
+				(font
+					(size 1.27 1.27)
+				)
+				(hide yes)
+			)
+		)
 		(pin "1"
 		)
@@
 			)
 		)
+		(property "Extra Value" ""
+			(at 139.7 78.74 0)
+			(effects
+				(font
+					(size 1.27 1.27)
+				)
+				(hide yes)
+			)
+		)
 		(pin "1"
 		)
@@
 			)
 		)
+		(property "Extra Value" ""
+			(at 116.84 71.12 0)
+			(effects
+				(font
+					(size 1.27 1.27)
+				)
+				(hide yes)
+			)
+		)
 		(pin "2"
 		)
@@
 			)
 		)
+		(property "Extra Value" ""
+			(at 172.72 68.58 0)
+			(effects
+				(font
+					(size 1.27 1.27)
+				)
+				(hide yes)
+			)
+		)
 		(pin "1"
 		)
@@
 		(in_bom no)
 		(on_board yes)
-		(dnp yes)
+		(dnp no)
 		(fields_autoplaced yes)
 		(property "Reference" "TP52"
@@
 			)
 		)
+		(property "Extra Value" ""
+			(at 127 149.86 0)
+			(effects
+				(font
+					(size 1.27 1.27)
+				)
+				(hide yes)
+			)
+		)
 		(pin "1"
 		)
@@
 					(bold yes)
 				)
+			)
+		)
+		(property "Extra Value" ""
+			(at 101.6 109.22 0)
+			(effects
+				(font
+					(size 1.27 1.27)
+				)
+				(hide yes)
 			)
 		)
@@
 			)
 		)
+		(property "Extra Value" ""
+			(at 101.6 78.74 0)
+			(effects
+				(font
+					(size 1.27 1.27)
+				)
+				(hide yes)
+			)
+		)
 		(pin "2"
 		)
@@
 		(in_bom no)
 		(on_board yes)
-		(dnp yes)
+		(dnp no)
 		(fields_autoplaced yes)
 		(property "Reference" "TP55"
@@
 			)
 		)
+		(property "Extra Value" ""
+			(at 127 38.1 0)
+			(effects
+				(font
+					(size 1.27 1.27)
+				)
+				(hide yes)
+			)
+		)
 		(pin "1"
 		)
@@
 		(in_bom no)
 		(on_board yes)
-		(dnp yes)
+		(dnp no)
 		(fields_autoplaced yes)
 		(property "Reference" "TP53"
@@
 			)
 		)
+		(property "Extra Value" ""
+			(at 127 165.1 0)
+			(effects
+				(font
+					(size 1.27 1.27)
+				)
+				(hide yes)
+			)
+		)
 		(pin "1"
 		)
@@
 			)
 		)
+		(property "Extra Value" ""
+			(at 172.72 137.16 0)
+			(effects
+				(font
+					(size 1.27 1.27)
+				)
+				(hide yes)
+			)
+		)
 		(pin "5"
 		)
@@
 			)
 		)
+		(property "Extra Value" ""
+			(at 83.82 71.12 0)
+			(effects
+				(font
+					(size 1.27 1.27)
+				)
+				(hide yes)
+			)
+		)
 		(pin "1"
 		)
@@
 		(in_bom no)
 		(on_board yes)
-		(dnp yes)
+		(dnp no)
 		(fields_autoplaced yes)
 		(property "Reference" "TP48"
@@
 			)
 		)
+		(property "Extra Value" ""
+			(at 88.9 43.18 0)
+			(effects
+				(font
+					(size 1.27 1.27)
+				)
+				(hide yes)
+			)
+		)

Commit message: workflow
Other:
- title: (none) -> Button, Status LED, UART, I2S
Changed lines of the file:
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@@
 	(generator_version "8.0")
 	(paper "A4")
+	(title_block
+		(title "Button, Status LED, UART, I2S")
+	)
 	(junction
 		(at 127 109.22)
