File: mcu.kicad_sch (KiCad schematic)
At the start: 10 parts, among them U1 ESP32-S3-WROOM-1U-N8

Commit message: commit before updating to LiveAstra lib
Parts:
- LED1: value 19-213/Y2C-CQ2R2L/3T(CY) -> LED_Yellow_25mA_0603
Connections:
- net IO_3_IC: now reaches R1.2, U1.15 (IO3)
Changed lines of the file:
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@@
+		)
+	)
+	(label "IO_3_IC"
+		(at 109.22 116.84 0)
+		(fields_autoplaced yes)
+		(effects
+			(font
+				(size 1.27 1.27)
+			)
+			(justify left bottom)
 		)
 	)
@@
 			)
 		)
-		(property "Value" "19-213/Y2C-CQ2R2L/3T(CY)"
+		(property "Value" "LED_Yellow_25mA_0603"
 			(at 238.76 55.88 0)
 			(effects

Commit message: Updated library name, updated and verified all footprints
Parts:
- C1: symbol EASYEDA2KICAD:C_22uF_X5R_0603 -> LiveAstra:C_22uF_X5R_0603
- C2, C3: symbol EASYEDA2KICAD:C_100nF_X7R_0402 -> LiveAstra:C_100nF_X7R_0402
- LED1: symbol EASYEDA2KICAD:LED_YELLOW_25mA_0603 -> LiveAstra:LED_YELLOW_25mA_0603
- R1: symbol EASYEDA2KICAD:R_0Ohm_0805_125mW -> LiveAstra:R_0Ohm_0805_125mW
- R2: symbol EASYEDA2KICAD:R_220Ohm_0402_62mW -> LiveAstra:R_220Ohm_0402_62mW
- TP1, TP2, TP3: symbol EASYEDA2KICAD:TestPoint_Thimble -> LiveAstra:TestPoint_Thimble
- U1: footprint EASYEDA2KICAD:WIRELM-SMD_ESP32-S3-WROOM-1U -> LiveAstra:WIRELM-SMD_ESP32-S3-WROOM-1U; symbol EASYEDA2KICAD:ESP32-S3-WROOM-1U-N8 -> LiveAstra:ESP32-S3-WROOM-1U-N8
Changed lines of the file:
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@@
 	)
 	(symbol
-		(lib_id "EASYEDA2KICAD:C_100nF_X7R_0402")
+		(lib_id "LiveAstra:C_100nF_X7R_0402")
 		(at 55.88 53.34 90)
 		(unit 1)
@@
 	)
 	(symbol
-		(lib_id "EASYEDA2KICAD:LED_YELLOW_25mA_0603")
+		(lib_id "LiveAstra:LED_YELLOW_25mA_0603")
 		(at 238.76 50.8 0)
 		(unit 1)
@@
 	)
 	(symbol
-		(lib_id "EASYEDA2KICAD:C_22uF_X5R_0603")
+		(lib_id "LiveAstra:C_22uF_X5R_0603")
 		(at 33.02 53.34 90)
 		(unit 1)
@@
 	)
 	(symbol
-		(lib_id "EASYEDA2KICAD:R_220Ohm_0402_62mW")
+		(lib_id "LiveAstra:R_220Ohm_0402_62mW")
 		(at 203.2 50.8 0)
 		(unit 1)
@@
 	)
 	(symbol
-		(lib_id "EASYEDA2KICAD:TestPoint_Thimble")
+		(lib_id "LiveAstra:TestPoint_Thimble")
 		(at 167.64 157.48 0)
 		(unit 1)
@@
 	)
 	(symbol
-		(lib_id "EASYEDA2KICAD:C_100nF_X7R_0402")
+		(lib_id "LiveAstra:C_100nF_X7R_0402")
 		(at 78.74 53.34 90)
 		(unit 1)
@@
 	)
 	(symbol
-		(lib_id "EASYEDA2KICAD:R_0Ohm_0805_125mW")
+		(lib_id "LiveAstra:R_0Ohm_0805_125mW")
 		(at 101.6 116.84 0)
 		(unit 1)
@@
 	)
 	(symbol
-		(lib_id "EASYEDA2KICAD:TestPoint_Thimble")
+		(lib_id "LiveAstra:TestPoint_Thimble")
 		(at 101.6 43.18 0)
 		(unit 1)
@@
 	)
 	(symbol
-		(lib_id "EASYEDA2KICAD:ESP32-S3-WROOM-1U-N8")
+		(lib_id "LiveAstra:ESP32-S3-WROOM-1U-N8")
 		(at 152.4 93.98 0)
 		(unit 1)
@@
 			)
 		)
-		(property "Footprint" "EASYEDA2KICAD:WIRELM-SMD_ESP32-S3-WROOM-1U"
+		(property "Footprint" "LiveAstra:WIRELM-SMD_ESP32-S3-WROOM-1U"
 			(at 152.4 171.45 0)
 			(effects
@@
 	)
 	(symbol
-		(lib_id "EASYEDA2KICAD:TestPoint_Thimble")
+		(lib_id "LiveAstra:TestPoint_Thimble")
 		(at 76.2 114.3 0)
 		(unit 1)

Commit message: Finished layout no drc or erc errors
Parts:
- removed TP2: TestPoint_Thimble, TestPoint:TestPoint_Loop_D3.50mm_Drill0.9mm_Beaded, symbol LiveAstra:TestPoint_Thimble
- C1: footprint Capacitor_SMD:C_0603_1608Metric -> LiveAstra:C_0603_1608Metric
- C2, C3: footprint Capacitor_SMD:C_0402_1005Metric -> LiveAstra:C_0402_1005Metric
- LED1: footprint LED_SMD:LED_0603_1608Metric -> LiveAstra:LED_0603_1608Metric
- R1: footprint Resistor_SMD:R_0805_2012Metric_Pad1.20x1.40mm_HandSolder -> LiveAstra:R_0805_2012Metric_Pad1.20x1.40mm_HandSolder
- R2: footprint Resistor_SMD:R_0402_1005Metric -> LiveAstra:R_0402_1005Metric
- TP1, TP3: footprint TestPoint:TestPoint_Loop_D3.50mm_Drill0.9mm_Beaded -> LiveAstra:TestPoint_Loop_D3.50mm_Drill0.9mm_Beaded; now not fitted; now left out of the parts list
Connections:
- net GPIO_12_BUTTON: now also U1.21 (IO13); no longer U1.20 (IO12)
- net GPIO_13_STATUS_LED: now also U1.20 (IO12); no longer U1.21 (IO13)
- net GPIO_14_I2S_WS: now also U1.23 (IO21); no longer U1.22 (IO14)
- net GPIO_15_RS485_DE: now also U1.5 (IO5); no longer U1.8 (IO15)
- net GPIO_15_RS485_RE: now also U1.6 (IO6); no longer U1.9 (IO16)
- net GPIO_17_RS485_TX: now also U1.4 (IO4); no longer U1.10 (IO17/U1_TX)
- net GPIO_18_RS485_RX: now also U1.7 (IO7); no longer U1.11 (IO18/U1_RX)
- net GPIO_21_I2S_SCK: now also U1.24 (IO47); no longer U1.23 (IO21)
- net GPIO_2_5V_OE: now also U1.39 (IO1); no longer U1.12 (IO8)
- net GPIO_35_5V: now also U1.35 (IO42); no longer U1.28 (IO35)
- net GPIO_36_5V: now also U1.34 (IO41); no longer U1.29 (IO36)
- net GPIO_37_5V: now also U1.33 (IO40); no longer U1.30 (IO37)
- net GPIO_38_5V: now also U1.32 (IO39); no longer U1.31 (IO38)
- net GPIO_39_PWM_CH1: now also U1.8 (IO15); no longer U1.32 (IO39)
- net GPIO_40_PWM_CH2: now also U1.11 (IO18); no longer U1.33 (IO40)
- net GPIO_41_PWM_CH3: now also U1.10 (IO17); no longer U1.34 (IO41)
- net GPIO_42_PWM_CH4: now also U1.9 (IO16); no longer U1.35 (IO42)
- net GPIO_47_I2S_SD: now also U1.25 (IO48); no longer U1.24 (IO47)
- net GPIO_48_I2S_LR: now also U1.22 (IO14); no longer U1.25 (IO48)
- net GPIO_4_FAN_TACHO: now also U1.29 (IO36); no longer U1.4 (IO4)
- net GPIO_5_FAN_PWM: now also U1.28 (IO35); no longer U1.5 (IO5)
- net GPIO_6_TEMP_I2C_SCL: now also U1.30 (IO37); no longer U1.6 (IO6)
- net GPIO_TEMP_I2C_SDA: now also U1.31 (IO38); no longer U1.7 (IO7)
- net IO_3_TEST: now reaches R1.1, TP1.1
Other:
- note added: "Update GPIO numbers!"
- moved on the sheet: LED1, R2

Commit message: Ready for kibot
Connections:
- net GPIO_12_BUTTON renamed GPIO_13_BUTTON
- net GPIO_13_STATUS_LED renamed GPIO_12_STATUS_LED
- net GPIO_14_I2S_WS renamed GPIO_21_I2S_WS
- net GPIO_15_RS485_DE renamed GPIO_5_RS485_DE
- net GPIO_15_RS485_RE renamed GPIO_6_RS485_RE
- net GPIO_17_RS485_TX renamed GPIO_4_RS485_TX
- net GPIO_18_RS485_RX renamed GPIO_7_RS485_RX
- net GPIO_21_I2S_SCK renamed GPIO_47_I2S_SCK
- net GPIO_2_5V_OE renamed GPIO_1_5V_OE
- net GPIO_35_5V renamed GPIO_42_5V
- net GPIO_36_5V renamed GPIO_41_5V
- net GPIO_37_5V renamed GPIO_40_5V
- net GPIO_38_5V renamed GPIO_39_5V
- net GPIO_39_PWM_CH1 renamed GPIO_15_PWM_CH4
- net GPIO_40_PWM_CH2 renamed GPIO_18_PWM_CH1
- net GPIO_41_PWM_CH3 renamed GPIO_17_PWM_CH2
- net GPIO_42_PWM_CH4 renamed GPIO_16_PWM_CH3
- net GPIO_47_I2S_SD renamed GPIO_48_I2S_SD
- net GPIO_48_I2S_LR renamed GPIO_14_I2S_LR
- net GPIO_4_FAN_TACHO renamed GPIO_36_FAN_TACHO
- net GPIO_5_FAN_PWM renamed GPIO_35_FAN_PWM
- net GPIO_6_TEMP_I2C_SCL renamed GPIO_37_TEMP_I2C_SCL
- net GPIO_TEMP_I2C_SDA renamed GPIO_38_TEMP_I2C_SDA
- net IO2_DEBUG_LED renamed GPIO_2_DEBUG_LED
- net IO2_DEBUG_LED_CL renamed GPIO_2_DEBUG_LED_CL

Commit message: workflow
Other:
- note removed: "Update GPIO numbers!"
Changed lines of the file:
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@@
-		)
-	)
-	(text "Update GPIO numbers!"
-		(exclude_from_sim no)
-		(at 195.58 111.76 0)
-		(effects
-			(font
-				(size 1.27 1.27)
-			)
 		)
 	)
@@
 	)
 	(hierarchical_label "GPIO_14_I2S_LR"
-		(shape bidirectional)
+		(shape output)
 		(at 182.88 137.16 0)
 		(fields_autoplaced yes)
@@
 	)
 	(hierarchical_label "GPIO_13_BUTTON"
-		(shape bidirectional)
+		(shape input)
 		(at 182.88 142.24 0)
 		(fields_autoplaced yes)
@@
 	)
 	(hierarchical_label "GPIO_18_PWM_CH1"
-		(shape bidirectional)
+		(shape output)
 		(at 121.92 91.44 180)
 		(fields_autoplaced yes)
@@
 	)
 	(hierarchical_label "GPIO_21_I2S_WS"
-		(shape bidirectional)
+		(shape output)
 		(at 182.88 132.08 0)
 		(fields_autoplaced yes)
@@
 	)
 	(hierarchical_label "GPIO_12_STATUS_LED"
-		(shape bidirectional)
+		(shape output)
 		(at 121.92 142.24 180)
 		(fields_autoplaced yes)
@@
 	)
 	(hierarchical_label "GPIO_37_TEMP_I2C_SCL"
-		(shape bidirectional)
+		(shape output)
 		(at 182.88 91.44 0)
 		(fields_autoplaced yes)
@@
 	)
 	(hierarchical_label "GPIO_48_I2S_SD"
-		(shape bidirectional)
+		(shape input)
 		(at 182.88 121.92 0)
 		(fields_autoplaced yes)
@@
 	)
 	(hierarchical_label "GPIO_47_I2S_SCK"
-		(shape bidirectional)
+		(shape output)
 		(at 182.88 127 0)
 		(fields_autoplaced yes)
@@
 	)
 	(hierarchical_label "GPIO_9_SCREEN_I2C_SCL"
-		(shape bidirectional)
+		(shape output)
 		(at 121.92 127 180)
 		(fields_autoplaced yes)
@@
 	)
 	(hierarchical_label "GPIO_36_FAN_TACHO"
-		(shape bidirectional)
+		(shape input)
 		(at 182.88 96.52 0)
 		(fields_autoplaced yes)

Commit message: workflow
Parts:
- U1: LCSC Part (none) -> C2980297
Changed lines of the file:
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@@
+			)
+		)
+		(property "LCSC Part" "C2980297"
+			(at 152.4 93.98 0)
+			(effects
+				(font
+					(size 1.27 1.27)
+				)
 			)
 		)

Commit message: workflow
Parts:
- TP1, TP3: now fitted
Changed lines of the file:
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@@
+			)
+		)
+		(property "Extra Value" ""
+			(at 55.88 53.34 0)
+			(effects
+				(font
+					(size 1.27 1.27)
+				)
+				(hide yes)
 			)
 		)
@@
 			)
 		)
+		(property "Extra Value" ""
+			(at 246.38 50.8 0)
+			(effects
+				(font
+					(size 1.27 1.27)
+				)
+				(hide yes)
+			)
+		)
 		(pin "1"
 		)
@@
 			)
 		)
+		(property "Extra Value" ""
+			(at 33.02 53.34 0)
+			(effects
+				(font
+					(size 1.27 1.27)
+				)
+				(hide yes)
+			)
+		)
 		(pin "2"
 		)
@@
 			)
 		)
+		(property "Extra Value" ""
+			(at 210.82 50.8 0)
+			(effects
+				(font
+					(size 1.27 1.27)
+				)
+				(hide yes)
+			)
+		)
 		(pin "1"
 		)
@@
 		(in_bom no)
 		(on_board yes)
-		(dnp yes)
+		(dnp no)
 		(fields_autoplaced yes)
 		(property "Reference" "TP3"
@@
 			)
 		)
+		(property "Extra Value" ""
+			(at 167.64 157.48 0)
+			(effects
+				(font
+					(size 1.27 1.27)
+				)
+				(hide yes)
+			)
+		)
 		(pin "1"
 		)
@@
 			)
 		)
+		(property "Extra Value" ""
+			(at 78.74 53.34 0)
+			(effects
+				(font
+					(size 1.27 1.27)
+				)
+				(hide yes)
+			)
+		)
 		(pin "1"
 		)
@@
 			)
 		)
+		(property "Extra Value" ""
+			(at 101.6 116.84 0)
+			(effects
+				(font
+					(size 1.27 1.27)
+				)
+				(hide yes)
+			)
+		)
 		(pin "1"
 		)
@@
 			)
 		)
+		(property "Extra Value" ""
+			(at 152.4 93.98 0)
+			(effects
+				(font
+					(size 1.27 1.27)
+				)
+				(hide yes)
+			)
+		)
 		(pin "11"
 		)
@@
 		(in_bom no)
 		(on_board yes)
-		(dnp yes)
+		(dnp no)
 		(fields_autoplaced yes)
 		(property "Reference" "TP1"
@@
 			)
 		)
+		(property "Extra Value" ""
+			(at 76.2 114.3 0)
+			(effects
+				(font
+					(size 1.27 1.27)
+				)
+				(hide yes)
+			)
+		)

Commit message: workflow
Other:
- title: (none) -> MCU
Changed lines of the file:
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@@
 	(generator_version "8.0")
 	(paper "A4")
+	(title_block
+		(title "MCU")
+	)
 	(junction
 		(at 167.64 160.02)
