File: overview.kicad_sch (KiCad schematic)
At the start: 0 parts

Commit message: workflow
Other:
- title: (none) -> Overview
Changed lines of the file:
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@@
 	(generator_version "8.0")
 	(paper "A4")
+	(title_block
+		(title "Overview")
+	)
 	(polyline
 		(pts
