File: usb.kicad_sch (KiCad schematic)
At the start: 7 parts, among them U4 USBLC6

Commit message: commit before updating to LiveAstra lib
Parts:
- USBC1: footprint Connector_USB:USB_C_Receptacle_HRO_TYPE-C-31-M-12 -> EASYEDA2KICAD:USB_C_Korean_Hroparts_Elec_TYPE-C-31-M-12
Changed lines of the file:
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@@
 			)
 		)
-		(property "Footprint" "Connector_USB:USB_C_Receptacle_HRO_TYPE-C-31-M-12"
+		(property "Footprint" "EASYEDA2KICAD:USB_C_Korean_Hroparts_Elec_TYPE-C-31-M-12"
 			(at 96.52 181.61 0)
 			(effects

Commit message: Updated library name, updated and verified all footprints
Parts:
- R12, R13: symbol EASYEDA2KICAD:R_5k1Ohm_0402_62mW -> LiveAstra:R_5k1Ohm_0402_62mW
- TP20, TP21, TP22: symbol EASYEDA2KICAD:TestPoint_Thimble -> LiveAstra:TestPoint_Thimble
- U4: footprint Package_TO_SOT_SMD:SOT-23-6 -> LiveAstra:USBLC6-4SC6_PROTECTION; symbol EASYEDA2KICAD:U_USBLC6_USB_TVS_ESD_SOT23_6L -> LiveAstra:U_USBLC6_USB_TVS_ESD_SOT23_6L
- USBC1: footprint EASYEDA2KICAD:USB_C_Korean_Hroparts_Elec_TYPE-C-31-M-12 -> LiveAstra:USB_C_Korean_Hroparts_Elec_TYPE-C-31-M-12; symbol EASYEDA2KICAD:USB_C_5A_Female_16PIN -> LiveAstra:USB_C_5A_Female_16PIN
Changed lines of the file:
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@@
 	)
 	(symbol
-		(lib_id "EASYEDA2KICAD:USB_C_5A_Female_16PIN")
+		(lib_id "LiveAstra:USB_C_5A_Female_16PIN")
 		(at 96.52 104.14 0)
 		(unit 1)
@@
 			)
 		)
-		(property "Footprint" "EASYEDA2KICAD:USB_C_Korean_Hroparts_Elec_TYPE-C-31-M-12"
+		(property "Footprint" "LiveAstra:USB_C_Korean_Hroparts_Elec_TYPE-C-31-M-12"
 			(at 96.52 181.61 0)
 			(effects
@@
 	)
 	(symbol
-		(lib_id "EASYEDA2KICAD:TestPoint_Thimble")
+		(lib_id "LiveAstra:TestPoint_Thimble")
 		(at 152.4 55.88 0)
 		(unit 1)
@@
 	)
 	(symbol
-		(lib_id "EASYEDA2KICAD:R_5k1Ohm_0402_62mW")
+		(lib_id "LiveAstra:R_5k1Ohm_0402_62mW")
 		(at 142.24 83.82 90)
 		(unit 1)
@@
 	)
 	(symbol
-		(lib_id "EASYEDA2KICAD:U_USBLC6_USB_TVS_ESD_SOT23_6L")
+		(lib_id "LiveAstra:U_USBLC6_USB_TVS_ESD_SOT23_6L")
 		(at 179.07 109.22 0)
 		(unit 1)
@@
 			)
 		)
-		(property "Footprint" "Package_TO_SOT_SMD:SOT-23-6"
+		(property "Footprint" "LiveAstra:USBLC6-4SC6_PROTECTION"
 			(at 179.07 146.05 0)
 			(effects
@@
 	)
 	(symbol
-		(lib_id "EASYEDA2KICAD:TestPoint_Thimble")
+		(lib_id "LiveAstra:TestPoint_Thimble")
 		(at 195.58 109.22 0)
 		(unit 1)
@@
 	)
 	(symbol
-		(lib_id "EASYEDA2KICAD:TestPoint_Thimble")
+		(lib_id "LiveAstra:TestPoint_Thimble")
 		(at 215.9 119.38 0)
 		(unit 1)
@@
 	)
 	(symbol
-		(lib_id "EASYEDA2KICAD:R_5k1Ohm_0402_62mW")
+		(lib_id "LiveAstra:R_5k1Ohm_0402_62mW")
 		(at 121.92 83.82 90)
 		(unit 1)
@@
 	)
 	(symbol
-		(lib_id "EASYEDA2KICAD:CHASSIS")
+		(lib_id "LiveAstra:CHASSIS")
 		(at 91.44 165.1 0)
 		(unit 1)

Commit message: Finished layout no drc or erc errors
Parts:
- removed U4: USBLC6, LiveAstra:USBLC6-4SC6_PROTECTION, symbol LiveAstra:U_USBLC6_USB_TVS_ESD_SOT23_6L
- added C27: 100n, LiveAstra:C_0402_1005Metric, symbol LiveAstra:C_100nF_X7R_0402
- added U7: USBLC6-2SC6, LiveAstra:USBLC6-2SC6_PROTECTION_SOT-23-6, symbol LiveAstra:U_USBLC6-2SC6_USB_TVS_ESD
- R12, R13: footprint Resistor_SMD:R_0402_1005Metric -> LiveAstra:R_0402_1005Metric
- TP13: renamed from TP20; footprint TestPoint:TestPoint_Loop_D3.50mm_Drill0.9mm_Beaded -> LiveAstra:TestPoint_Loop_D3.50mm_Drill0.9mm_Beaded; now not fitted; now left out of the parts list
- TP14: renamed from TP21; footprint TestPoint:TestPoint_Loop_D3.50mm_Drill0.9mm_Beaded -> LiveAstra:TestPoint_Loop_D3.50mm_Drill0.9mm_Beaded; now not fitted; now left out of the parts list
- TP15: renamed from TP22; footprint TestPoint:TestPoint_Loop_D3.50mm_Drill0.9mm_Beaded -> LiveAstra:TestPoint_Loop_D3.50mm_Drill0.9mm_Beaded; now not fitted; now left out of the parts list
Connections:
- net GND: now also C27.1, U7.2 (GND)
- net VBUS: now also C27.2, U7.5 (VBUS)
- net D+ renamed USB_CONN_D+
- net USB_CONN_D+: now also U7.3 (USB_IN_D+); no longer TP15.1
- net D- renamed USB_CONN_D-
- net USB_CONN_D-: now also U7.1 (USB_IN_D-); no longer TP14.1
- new net USB_D+: TP15.1, U7.4 (USB_OUT_D+)
- new net USB_D-: TP14.1, U7.6 (USB_OUT_D-)

Commit message: Work on kibot
Parts:
- R12, R13: Extra Values 50V ±1% 0402 62.5mW -> 50V ±1% 0402 62.5mW

Commit message: workflow
Parts:
- TP13, TP14, TP15: now fitted
Changed lines of the file:
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@@
+			)
+		)
+		(property "Extra Value" ""
+			(at 96.52 104.14 0)
+			(effects
+				(font
+					(size 1.27 1.27)
+				)
+				(hide yes)
 			)
 		)
@@
 		(in_bom no)
 		(on_board yes)
-		(dnp yes)
+		(dnp no)
 		(fields_autoplaced yes)
 		(property "Reference" "TP13"
@@
 			)
 		)
+		(property "Extra Value" ""
+			(at 152.4 55.88 0)
+			(effects
+				(font
+					(size 1.27 1.27)
+				)
+				(hide yes)
+			)
+		)
 		(pin "1"
 		)
@@
 			)
 		)
+		(property "Extra Value" ""
+			(at 142.24 83.82 0)
+			(effects
+				(font
+					(size 1.27 1.27)
+				)
+				(hide yes)
+			)
+		)
 		(pin "1"
 		)
@@
 			)
 		)
+		(property "Extra Value" ""
+			(at 193.04 66.04 0)
+			(effects
+				(font
+					(size 1.27 1.27)
+				)
+				(hide yes)
+			)
+		)
 		(pin "1"
 		)
@@
 		(in_bom no)
 		(on_board yes)
-		(dnp yes)
+		(dnp no)
 		(fields_autoplaced yes)
 		(property "Reference" "TP14"
@@
 			)
 		)
+		(property "Extra Value" ""
+			(at 203.2 109.22 0)
+			(effects
+				(font
+					(size 1.27 1.27)
+				)
+				(hide yes)
+			)
+		)
 		(pin "1"
 		)
@@
 			)
 		)
+		(property "Extra Value" ""
+			(at 177.8 109.22 0)
+			(effects
+				(font
+					(size 1.27 1.27)
+				)
+				(hide yes)
+			)
+		)
 		(pin "5"
 		)
@@
 		(in_bom no)
 		(on_board yes)
-		(dnp yes)
+		(dnp no)
 		(fields_autoplaced yes)
 		(property "Reference" "TP15"
@@
 			)
 		)
+		(property "Extra Value" ""
+			(at 203.2 119.38 0)
+			(effects
+				(font
+					(size 1.27 1.27)
+				)
+				(hide yes)
+			)
+		)
 		(pin "1"
 		)
@@
 			)
 		)
+		(property "Extra Value" ""
+			(at 121.92 83.82 0)
+			(effects
+				(font
+					(size 1.27 1.27)
+				)
+				(hide yes)
+			)
+		)

Commit message: workflow
Other:
- title: (none) -> USB
Changed lines of the file:
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@@
 	(generator_version "8.0")
 	(paper "A4")
+	(title_block
+		(title "USB")
+	)
 	(junction
 		(at 127 58.42)
