File: AstraControlPCB/5V_Protection.kicad_sch (KiCad schematic)
At the start: 8 parts, among them U2 NCP361SNT1G

Commit message: Update wks file
Other:
- company: (none) -> LiveAstra Technologies
- title: 5V Protection -> AstraControl - Root
Changed lines of the file:
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@@
 	(paper "A4")
 	(title_block
-		(title "5V Protection")
+		(title "AstraControl - Root")
+		(date "2024-08-26")
+		(rev "A")
+		(company "LiveAstra Technologies")
 	)
 	(junction
@@
 		(effects
 			(font
-				(face "Sarabun")
+				(face "ING Me")
 				(size 3 3)
 				(color 255 255 255 1)
@@
 		(effects
 			(font
+				(face "ING Me")
 				(size 1.5 1.5)
 				(color 255 255 255 1)
@@
 		)
 		(instances
-			(project ""
+			(project "AstraControl"
 				(path "/9a751838-dce8-4d69-8a02-736625ac74e7/0db21d8e-3390-4d67-877f-0e5d98e37848/e21714b4-6921-40f8-8882-480f43314016"
 					(reference "R8")
