File: AstraControlPCB/AstraControl.kicad_sch (KiCad schematic)
At the start: 0 parts

Commit message: Update wks file
Other:
- title: AstraControl - ESP32 Based Controller -> AstraControl - Root
Changed lines of the file:
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@@
 	(paper "A4")
 	(title_block
-		(title "AstraControl - ESP32 Based Controller")
+		(title "AstraControl - Root")
+		(date "2024-08-26")
 		(rev "A")
 		(company "LiveAstra Technologies")
@@
 		(effects
 			(font
+				(face "ING Me")
 				(size 3 3)
 			)
@@
 		(effects
 			(font
-				(face "Sarabun SemiBold")
+				(face "ING Me")
 				(size 4 4)
 				(thickness 0.8)
@@
 		(effects
 			(font
+				(face "ING Me")
 				(size 3 3)
 			)
@@
 		(effects
 			(font
+				(face "ING Me")
 				(size 3 3)
 			)
@@
 		(effects
 			(font
-				(face "Sarabun ExtraBold")
+				(face "ING Me")
 				(size 5 5)
 				(color 255 255 255 1)
@@
 		(effects
 			(font
+				(face "ING Me")
 				(size 3 3)
 			)
@@
 		(effects
 			(font
+				(face "ING Me Headline")
 				(size 8 8)
 				(thickness 1.6)
@@
 		(effects
 			(font
+				(face "ING Me")
 				(size 3 3)
 			)
@@
 		(effects
 			(font
+				(face "ING Me")
 				(size 3 3)
 			)
@@
 		(effects
 			(font
+				(face "ING Me")
 				(size 5 5)
 			)
@@
 		(effects
 			(font
+				(face "ING Me")
 				(size 3 3)
 			)
@@
 		(effects
 			(font
+				(face "ING Me")
 				(size 3 3)
 			)
@@
 		(effects
 			(font
-				(face "Sarabun")
+				(face "ING Me")
 				(size 3 3)
 				(color 255 255 255 1)
@@
 		(effects
 			(font
-				(face "Sarabun")
+				(face "ING Me")
 				(size 3 3)
 				(color 255 255 255 1)
@@
 		(effects
 			(font
-				(face "Sarabun")
+				(face "ING Me")
 				(size 3 3)
 				(color 255 255 255 1)
@@
 		(effects
 			(font
+				(face "ING Me")
 				(size 4 4)
 			)
@@
 		(effects
 			(font
+				(face "ING Me")
 				(size 3 3)
 			)
@@
 		(effects
 			(font
-				(face "Sarabun")
+				(face "ING Me")
 				(size 3 3)
 				(color 255 255 255 1)
@@
 	)
 	(sheet
-		(at 106 157)
+		(at 114.89 151.92)
 		(size 34 27)
 		(fields_autoplaced yes)
@@
 		)
 		(property "Sheetname" "Block Diagram"
-			(at 106 156.2884 0)
+			(at 114.89 151.2084 0)
 			(effects
 				(font
@@
 		)
 		(property "Sheetfile" "block_diagram.kicad_sch"
-			(at 106 184.5846 0)
+			(at 114.89 179.5046 0)
 			(effects
 				(font
@@
 	)
 	(sheet
-		(at 52 158)
+		(at 63.43 152.92)
 		(size 34 24)
 		(fields_autoplaced yes)
@@
 		)
 		(property "Sheetname" "Overview"
-			(at 52 157.2884 0)
+			(at 63.43 152.2084 0)
 			(effects
 				(font
@@
 		)
 		(property "Sheetfile" "overview.kicad_sch"
-			(at 52 182.5846 0)
+			(at 63.43 177.5046 0)
 			(effects
 				(font

Commit message: workflow
Other:
- note added: "2x 5V GPIO"
- note added: "2x I2C Auxilary"
- note added: "4 Channel LED PWM"
- note added: "4 Wire 5V Fan"
- note added: "5V to 3.3V Step Down DC-DC"
- note added: "ESP32-S3 SoC integrating Wi-Fi 4 and Bluetooth 5 (LE)"
- note added: "ESP32-based control PCB uses WiFi with an external antenna and 5Mbps RS-485 for communication, supporting various sensors and HMI devices for high-power LED fixtures or strips."
- note added: "External button and status LED"
- note added: "I2S"
- note added: "UART"
- note added: "Up to 5V 10A Input"
- note removed: "-"
- note removed: "5V 10A Input"
- note removed: "Button"
- note removed: "ESP32"
- note removed: "ESP32 Based control PCB for other light fixture pcbs."
- note removed: "GPIO Breakout"
- note removed: "I2C Auxilary"

Commit message: workflow
Changed lines of the file:
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@@
-		)
-	)
-	(rectangle
-		(start 20.32 123.19)
-		(end 29.21 128.27)
-		(stroke
-			(width 0)
-			(type default)
-		)
-		(fill
-			(type none)
-		)
-	)
-	(rectangle
-		(start 20.32 129.54)
-		(end 29.21 134.62)
-		(stroke
-			(width 0)
-			(type default)
-		)
-		(fill
-			(type none)
 		)
 	)
@@
 	)
 	(rectangle
-		(start 182.5 67.5)
-		(end 277.5 155)
+		(start 196.85 76.2)
+		(end 279.4 139.7)
 		(stroke
 			(width 0)
@@
 		)
 	)
-	(rectangle
-		(start 20.32 104.14)
-		(end 29.21 109.22)
-		(stroke
-			(width 0)
-			(type default)
-		)
-		(fill
-			(type none)
-		)
-	)
-	(rectangle
-		(start 20.32 116.84)
-		(end 29.21 121.92)
-		(stroke
-			(width 0)
-			(type default)
-		)
-		(fill
-			(type none)
-		)
-	)
 	(circle
 		(center 21.59 125.73)
@@
 		)
 	)
-	(rectangle
-		(start 20.32 148.59)
-		(end 29.21 153.67)
-		(stroke
-			(width 0)
-			(type default)
-		)
-		(fill
-			(type none)
-		)
-	)
-	(rectangle
-		(start 20.32 91.44)
-		(end 29.21 96.52)
-		(stroke
-			(width 0)
-			(type default)
-		)
-		(fill
-			(type none)
-		)
-	)
 	(circle
 		(center 21.59 106.68)
@@
 		)
 	)
-	(rectangle
-		(start 20.32 142.24)
-		(end 29.21 147.32)
-		(stroke
-			(width 0)
-			(type default)
-		)
-		(fill
-			(type none)
-		)
-	)
-	(rectangle
-		(start 20.32 110.49)
-		(end 29.21 115.57)
-		(stroke
-			(width 0)
-			(type default)
-		)
-		(fill
-			(type none)
-		)
-	)
 	(circle
 		(center 21.59 113.03)
@@
 		)
 	)
-	(rectangle
-		(start 20.32 154.94)
-		(end 29.21 160.02)
-		(stroke
-			(width 0)
-			(type default)
-		)
-		(fill
-			(type none)
-		)
-	)
 	(circle
 		(center 21.59 157.48)
@@
 		)
 	)
-	(rectangle
-		(start 20.32 85.09)
-		(end 29.21 90.17)
-		(stroke
-			(width 0)
-			(type default)
-		)
-		(fill
-			(type none)
-		)
-	)
 	(circle
 		(center 21.59 151.13)
@@
 		)
 	)
-	(rectangle
-		(start 20.32 97.79)
-		(end 29.21 102.87)
-		(stroke
-			(width 0)
-			(type default)
-		)
-		(fill
-			(type none)
-		)
-	)
-	(rectangle
-		(start 20.32 161.29)
-		(end 29.21 166.37)
-		(stroke
-			(width 0)
-			(type default)
-		)
-		(fill
-			(type none)
-		)
-	)
 	(circle
 		(center 21.59 163.83)
@@
 		)
 	)
-	(rectangle
-		(start 20.32 135.89)
-		(end 29.21 140.97)
-		(stroke
-			(width 0)
-			(type default)
-		)
-		(fill
-			(type none)
-		)
-	)
 	(circle
 		(center 21.59 138.43)
@@
 	(text "Render placeholder"
 		(exclude_from_sim no)
-		(at 205 115 0)
+		(at 215.9 107.95 0)
 		(effects
 			(font
@@
 	(text "In review"
 		(exclude_from_sim no)
-		(at 31.75 44.45 0)
-		(effects
-			(font
-				(face "ING Me")
-				(size 5 5)
+		(at 30.48 40.64 0)
+		(effects
+			(font
+				(face "ING Me")
+				(size 4.064 4.064)
 			)
 		)
@@
 	(text "Features"
 		(exclude_from_sim no)
-		(at 19.05 82.55 0)
+		(at 19.05 81.28 0)
 		(effects
 			(font
 				(face "ING Me")
 				(size 4 4)
+				(thickness 0.8)
+				(bold yes)
 			)
 			(justify left)
@@
 	)
 	(sheet
-		(at 114.89 151.92)
-		(size 34 27)
+		(at 241.89 145.57)
+		(size 37.51 32.23)
 		(fields_autoplaced yes)
 		(stroke
@@
 		)
 		(property "Sheetname" "Block Diagram"
-			(at 114.89 151.2084 0)
+			(at 241.89 144.8584 0)
 			(effects
 				(font
@@
 		)
 		(property "Sheetfile" "block_diagram.kicad_sch"
-			(at 114.89 179.5046 0)
+			(at 241.89 178.3846 0)
 			(effects
 				(font
@@
 	)
 	(sheet
-		(at 63.43 152.92)
-		(size 34 24)
+		(at 196.85 146.05)
+		(size 38.1 31.75)
 		(fields_autoplaced yes)
 		(stroke
@@
 		)
 		(property "Sheetname" "Overview"
-			(at 63.43 152.2084 0)
+			(at 196.85 145.3384 0)
 			(effects
 				(font
@@
 		)
 		(property "Sheetfile" "overview.kicad_sch"
-			(at 63.43 177.5046 0)
+			(at 196.85 178.3846 0)
 			(effects
 				(font

Commit message: workflow
Other:
- note added: "Render for reference only"
- note removed: "Render placeholder"

Commit message: workflow
Other:
- note added: "ESP32-based control PCB uses WiFi with an external antenna and 5Mbps RS-485 for communication, supporting various sensors and HMI devices for high-power LED fixtures or strips. One device can act as master or all fixtures will receive data from a dedicated receiver."
- note removed: "ESP32-based control PCB uses WiFi with an external antenna and 5Mbps RS-485 for communication, supporting various sensors and HMI devices for high-power LED fixtures or strips."
Changed lines of the file:
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@@
 		(fill
 			(type color)
-			(color 255 255 255 1)
+			(color 0 0 0 0)
 		)
 	)
 	(circle
-		(center 21.59 93.98)
-		(radius 0.6174)
+		(center 21.59 144.78)
+		(radius 0.82)
 		(stroke
 			(width -0.0001)
@@
 		(fill
 			(type color)
-			(color 255 255 255 1)
+			(color 0 0 0 0)
 		)
 	)
 	(circle
-		(center 21.59 144.78)
-		(radius 0.7071)
+		(center 21.59 93.98)
+		(radius 0.6174)
 		(stroke
 			(width -0.0001)
@@
 		(fill
 			(type color)
-			(color 255 255 255 1)
+			(color 0 0 0 0)
 		)
 	)
@@
 		(fill
 			(type color)
-			(color 255 255 255 1)
+			(color 0 0 0 0)
 		)
 	)
 	(circle
-		(center 21.59 106.68)
-		(radius 0.6696)
+		(center 21.59 151.13)
+		(radius 0.82)
 		(stroke
 			(width -0.0001)
@@
 		(fill
 			(type color)
-			(color 255 255 255 1)
+			(color 0 0 0 0)
 		)
 	)
 	(circle
-		(center 21.59 113.03)
-		(radius 0.73)
+		(center 21.59 106.68)
+		(radius 0.6696)
 		(stroke
 			(width -0.0001)
@@
 		(fill
 			(type color)
-			(color 255 255 255 1)
+			(color 0 0 0 0)
 		)
 	)
 	(circle
-		(center 21.59 100.33)
-		(radius 0.6306)
+		(center 21.59 113.03)
+		(radius 0.73)
 		(stroke
 			(width -0.0001)
@@
 		(fill
 			(type color)
-			(color 255 255 255 1)
+			(color 0 0 0 0)
 		)
 	)
 	(circle
-		(center 21.59 157.48)
-		(radius 0.82)
+		(center 21.59 100.33)
+		(radius 0.6306)
 		(stroke
 			(width -0.0001)
@@
 		(fill
 			(type color)
-			(color 255 255 255 1)
+			(color 0 0 0 0)
 		)
 	)
@@
 		(fill
 			(type color)
-			(color 255 255 255 1)
+			(color 0 0 0 0)
 		)
 	)
 	(circle
-		(center 21.59 151.13)
+		(center 21.59 157.48)
 		(radius 0.82)
 		(stroke
@@
 		(fill
 			(type color)
-			(color 255 255 255 1)
+			(color 0 0 0 0)
 		)
 	)
@@
 		(fill
 			(type color)
-			(color 255 255 255 1)
+			(color 0 0 0 0)
 		)
 	)
@@
 		(fill
 			(type color)
-			(color 255 255 255 1)
+			(color 0 0 0 0)
 		)
 	)
@@
 		(fill
 			(type color)
-			(color 255 255 255 1)
+			(color 0 0 0 0)
 		)
 	)
@@
 				(face "ING Me")
 				(size 3 3)
-				(color 255 255 255 1)
 			)
 			(justify left)
@@
 		)
 	)
-	(text "ESP32-based control PCB uses WiFi with an external antenna and 5Mbps RS-485\nfor communication, supporting various sensors and HMI devices for high-power \nLED fixtures or strips."
+	(text "ESP32-based control PCB uses WiFi with an external antenna and 5Mbps RS-485\nfor communication, supporting various sensors and HMI devices for high-power \nLED fixtures or strips. One device can act as master or all fixtures will receive \ndata from a dedicated receiver."
 		(exclude_from_sim no)
 		(at 19.05 63.5 0)
@@
 				(face "ING Me")
 				(size 3 3)
-				(color 255 255 255 1)
 			)
 			(justify left)
@@
 				(face "ING Me")
 				(size 3 3)
-				(color 255 255 255 1)
 			)
 			(justify left)
@@
 				(face "ING Me")
 				(size 3 3)
-				(color 255 255 255 1)
 			)
 			(justify left)
@@
 				(face "ING Me")
 				(size 3 3)
-				(color 255 255 255 1)
 			)
 			(justify left)
