File: AstraControlPCB/fan_temp_screen.kicad_sch (KiCad schematic)
At the start: 22 parts, among them CN4 4P JST ZH, CN5 4P JST ZH, CN6 4P JST ZH

Commit message: Update wks file
Other:
- company: (none) -> LiveAstra Technologies
- title: Fan, Temperature and Screen -> AstraControl - Root
Changed lines of the file:
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@@
 	(paper "A4")
 	(title_block
-		(title "Fan, Temperature and Screen")
+		(title "AstraControl - Root")
+		(date "2024-08-26")
+		(rev "A")
+		(company "LiveAstra Technologies")
 	)
 	(junction
@@
 		(effects
 			(font
+				(face "ING Me")
 				(size 1.5 1.5)
 				(color 255 255 255 1)
@@
 		(effects
 			(font
-				(face "Sarabun")
+				(face "ING Me")
 				(size 3 3)
 				(color 255 255 255 1)

Commit message: Remove plus minus symbol
Parts:
- C21: Extra Values 50V C0G ±5% 0805 -> 50V C0G 5% 0805
- R23, R24, R28, R30: Extra Values 50V ±1% 0402 62.5mW -> 50V 1% 0402 62.5mW
- R25, R26, R43, R44, R45, R46: Extra Values 150V ±1% 0805 -> 150V 1% 0805
- R27: Extra Values 50V ±1% 0402 62mW -> 50V 1% 0402 62mW
- R29: Extra Values 150V ±1% 0805 125mW -> 150V 1% 0805 125mW

Commit message: workflow
Parts:
- added INF7: ~, symbol LiveAstra:Information_Box
Other:
- note added: "Fan Temperature Screen"
- note removed: "Cutoff frequency: 482kHz"
- note removed: "RC Filter"
- moved on the sheet: C21, CN4, CN5, CN6, R23, R24, R25, R26, R27, R28, R29, R30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

Commit message: update
Parts:
- renumbered C21 to C22, INF7 to INF6, R43 to R26, R46 to R27, R26 to R28, R27 to R29, R29 to R30, R30 to R31, R28 to R32, R44 to R33, R45 to R34, TP38 to TP33, TP37 to TP34, TP36 to TP35, TP39 to TP36, TP41 to TP37, TP40 to TP38

Commit message: update
Other:
- note added: "RC Filter Cutoff: 482KHz"
- moved on the sheet: C22, CN4, CN5, CN6, R23, R24, R25, R26, R27, R28, R29, R30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
