File: AstraControlPCB/AstraControl.kicad_pcb (KiCad board)
At the start: 4 copper layers, 102 x 96 mm, 153 parts, among them CN1 4P JST VH, CN10 JST_ZH_6PIN_1A_250V, CN2 4P JST VH, CN3 4P JST VH, CN4 4P JST ZH, CN5 4P JST ZH, CN6 4P JST ZH, CN7 JST_VH_8PIN_10A_250V, CN8 4P JST ZH, CN9 4P JST ZH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

Commit message: update
Parts:
- C12, C15, C17: value 47u -> DNP
- R26, R27, R33, R34: value 0 -> DNP
- R45, R46, R47: value 1M -> DNP

Commit message: update
Routing:
- net GND: vias 309 -> 308

Commit message: Another redesign
Parts:
- removed G1: ~, LiveAstra:AstraControl_Ground_Band
- removed kibuzzard-66D4B301: G***, kibuzzard-66D4B301
- added RING1: ~, LiveAstra:AstraControl_Ground_Ring, F.Cu at (149.8, 80.1)
- moved R44 64.7 mm to (100.0, 43.9), turned to 90 degrees
- moved R45 63.8 mm to (196.9, 44.6), turned to 90 degrees
- moved C24 62.9 mm to (100.0, 48.7), turned to 90 degrees
- moved C25 62.0 mm to (197.0, 49.4), turned to 90 degrees
- moved C27 57.6 mm to (100.0, 109.3), turned to 90 degrees
- moved R47 55.9 mm to (99.8, 104.6), turned to 90 degrees
- moved R46 54.3 mm to (196.3, 104.1)
- moved C26 54.0 mm to (196.4, 108.9), turned to 90 degrees
- moved TP11 40.3 mm to (100.0, 120.1)
- moved TP2 39.7 mm to (148.5, 89.1)
- moved TP10 34.0 mm to (104.8, 120.1)
- moved R33 25.3 mm to (129.3, 100.1), turned to 90 degrees
- moved R31 24.5 mm to (131.0, 99.3), turned to 90 degrees
- moved SW2 24.0 mm to (107.3, 94.2), turned to 0 degrees
- moved R6 20.9 mm to (103.3, 100.4), turned to -90 degrees
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Routing:
- net +3V3: track 256.7 -> 0.00 mm, vias 9 -> 0
- net /Block Diagram/Fan, Temperature and Screen/TEMP_I2C_SDA: track 74.5 -> 0.00 mm
- net GND: track 76.0 -> 4.59 mm, vias 308 -> 5
- net /Block Diagram/Fan, Temperature and Screen/TEMP_I2C_SCL: track 69.8 -> 0.00 mm
- net /Block Diagram/Fan, Temperature and Screen/SCREEN_I2C_SCL: track 65.5 -> 0.00 mm
- net /Block Diagram/Fan, Temperature and Screen/SCREEN_I2C_SDA: track 58.5 -> 0.00 mm
- net /Block Diagram/Button, Status LED, UART and I2S/I2S_SD: track 54.2 -> 0.00 mm
- net /Block Diagram/Button, Status LED, UART and I2S/I2S_SCK: track 51.7 -> 0.00 mm
- net /Block Diagram/Button, Status LED, UART and I2S/I2S_WS: track 49.7 -> 0.00 mm
- net /Block Diagram/Button, Status LED, UART and I2S/I2S_LR: track 49.5 -> 0.00 mm
- net /Block Diagram/MCU Enable and Boot/EN_DELAY: track 47.9 -> 0.00 mm, vias 2 -> 0
- net +5V_IN: track 45.5 -> 0.00 mm
- net /Block Diagram/Button, Status LED, UART and I2S/UART_TX: track 45.3 -> 0.00 mm, vias 1 -> 0
- net /Block Diagram/3V3 to 5V Logic Shifter/3V3_IO_1: track 44.7 -> 0.00 mm
- net /Block Diagram/3V3 to 5V Logic Shifter/3V3_IO_4: track 44.5 -> 0.00 mm
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- removed copper zone on F.Cu, net +3V3
- removed copper zone on F.Cu, net +5V
- removed copper zone on B.Cu, net +5V_IN
- removed copper zone on F.Cu, net +5V_IN
- removed copper zone on F.Cu, net /Block Diagram/5V to 3.3V/SW_OUT
- removed copper zone on F.Cu, net /Block Diagram/5V to 3.3V/SW_OUT_UNFILTERED
- removed copper zone on B.Cu, net CHASSIS
- removed copper zone on F.Cu, net CHASSIS
- removed copper zone on B.Cu, net GND
- removed copper zone on F.Cu, net GND
Other:
- board text removed: "10A Max"
- board text removed: "15"
- board text removed: "16"
- board text removed: "17"
- board text removed: "18"
- board text removed: "3V3"
- board text removed: "5V"
- board text removed: "5V IN"
- board text removed: "A"
- board text removed: "B"
- board text removed: "BTN"
- board text removed: "D+"
- board text removed: "D-"
- board text removed: "DE"
- board text removed: "DEBUG LED"
- board text removed: "EN"
- board text removed: "FAN"
- board text removed: "G"
- board text removed: "GND"
- board text removed: "IO0"
- board text removed: "IO15"
- board text removed: "IO16"
- board text removed: "IO17"
- board text removed: "IO18"
- board text removed: "IO3"
- board text removed: "IO39"
- board text removed: "IO40"
- board text removed: "IO41"
- board text removed: "IO42"
- board text removed: "JLCJLCJLCJLC"
- board text removed: "LED"
- board text removed: "LR"
- board text removed: "OE"
- board text removed: "PWR ON"
- board text removed: "RE"
- board text removed: "RESET"
- board text removed: "RX"
- board text removed: "SCK"
- board text removed: "SCL"
- board text removed: "SD"
- board text removed: "SDA"
- board text removed: "TCH"
- board text removed: "TX"
- board text removed: "VBUS"
- board text removed: "WS"
- board text removed: "[ ]"
- board text removed: "liveleds.io"
- board text removed: "~3V3"

Commit message: More routing
Parts:
- moved RING1 116.9 mm to (33.0, 82.1)
- moved CN5 16.5 mm to (184.3, 119.6), turned to 180 degrees
- moved TP35 16.5 mm to (167.8, 114.6)
- moved TP37 16.5 mm to (184.3, 114.6)
- moved TP48 13.5 mm to (150.8, 114.6)
- moved TP51 13.5 mm to (137.3, 114.6)
- moved R25 11.7 mm to (127.8, 100.1)
- moved R30 11.5 mm to (130.0, 100.1)
- moved C22 11.2 mm to (132.3, 100.2), turned to 90 degrees
- moved R33 10.2 mm to (139.5, 100.1), turned to 180 degrees
- moved R31 9.35 mm to (140.0, 101.9), turned to 180 degrees
- moved R28 8.88 mm to (130.0, 104.9)
- moved CN10 7.55 mm to (147.8, 119.6), turned to 180 degrees
- moved CN4 7.55 mm to (172.3, 119.6), turned to 180 degrees
- moved TP33 7.50 mm to (179.8, 114.6)
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Connections:
- net /Block Diagram/5V Protection/VBUS renamed /Block Diagram/Power Connectors/USB/VBUS
- USBC1 pad A8: unconnected-(USBC1-SBU1-PadA8) -> (no net)
- USBC1 pad B8: unconnected-(USBC1-SBU2-PadB8) -> (no net)
Routing:
- net /Block Diagram/Fan, Temperature and Screen/TEMP_I2C_SDA: track 0.00 -> 75.0 mm
- net /Block Diagram/Fan, Temperature and Screen/TEMP_I2C_SCL: track 0.00 -> 73.2 mm
- net /Block Diagram/Button, Status LED, UART and I2S/I2S_SD: track 0.00 -> 61.8 mm, vias 0 -> 2
- net /Block Diagram/Button, Status LED, UART and I2S/I2S_SCK: track 0.00 -> 58.9 mm, vias 0 -> 2
- net /Block Diagram/Button, Status LED, UART and I2S/I2S_LR: track 0.00 -> 57.3 mm, vias 0 -> 2
- net /Block Diagram/Button, Status LED, UART and I2S/I2S_WS: track 0.00 -> 56.8 mm, vias 0 -> 2
- net /Block Diagram/Fan, Temperature and Screen/FAN_PWM_CON: track 0.00 -> 55.2 mm
- net /Block Diagram/Fan, Temperature and Screen/FAN_TACHO_CON: track 0.00 -> 54.3 mm
- net /Block Diagram/Fan, Temperature and Screen/SCREEN_I2C_SDA: track 0.00 -> 51.9 mm
- net /Block Diagram/Fan, Temperature and Screen/SCREEN_I2C_SCL: track 0.00 -> 51.1 mm
- net /Block Diagram/Button, Status LED, UART and I2S/UART_TX: track 0.00 -> 43.8 mm, vias 0 -> 2
- net /Block Diagram/Button, Status LED, UART and I2S/UART_RX: track 0.00 -> 40.7 mm, vias 0 -> 2
- net /Block Diagram/Button, Status LED, UART and I2S/STATUS_LED: track 0.00 -> 29.6 mm
- net /Block Diagram/Button, Status LED, UART and I2S/BUTTON: track 0.00 -> 27.9 mm
- net /Block Diagram/LED PWM Connector/PWM_CH4: track 21.1 -> 0.00 mm
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
Commit message: Updates
Parts:
- added R48: DNP, LiveAstra:R_0805_2012Metric_Pad1.20x1.40mm_HandSolder, F.Cu at (151.5, 58.6)
- added R49: DNP, LiveAstra:R_0805_2012Metric_Pad1.20x1.40mm_HandSolder, F.Cu at (150.0, 67.1)
- moved RING1 117.3 mm to (150.2, 79.6)
- moved TP27 16.9 mm to (158.5, 73.4)
- moved TP8 12.8 mm to (172.5, 109.6)
- moved TP22 12.3 mm to (158.5, 86.9)
- moved TP1 11.1 mm to (117.0, 68.1)
- moved TP11 10.6 mm to (107.0, 112.1)
- moved C15 10.3 mm to (157.0, 94.1), turned to 180 degrees
- moved TP9 10.2 mm to (152.8, 95.4)
- moved R18 9.80 mm to (151.0, 61.6), turned to 0 degrees
- moved R19 9.78 mm to (151.0, 64.1)
- moved TP2 8.98 mm to (138.8, 83.1)
- moved R39 8.86 mm to (133.8, 60.1)
- moved R20 8.73 mm to (149.8, 59.1), turned to 90 degrees
- moved TP28 8.43 mm to (177.5, 73.4)
- moved TP24 7.27 mm to (158.5, 77.9)
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Connections:
- net /Block Diagram/LED PWM Connector/EXTRA_PIN renamed /Block Diagram/LED PWM Connector/RESERVED_PIN
Routing:
- net +3V3: track 0.96 -> 103.4 mm, vias 1 -> 12
- net /Block Diagram/MCU Enable and Boot/EN_DELAY: track 0.00 -> 51.8 mm, vias 0 -> 2
- net /Block Diagram/3V3 to 5V Logic Shifter/3V3_IO_1: track 10.4 -> 49.1 mm
- net /Block Diagram/MCU/GPIO_6_RS485_RE: track 0.00 -> 38.1 mm, vias 0 -> 3
- net /Block Diagram/MCU/GPIO_5_RS485_DE: track 0.00 -> 35.8 mm, vias 0 -> 3
- net /Block Diagram/3V3 to 5V Logic Shifter/3V3_IO_2: track 12.8 -> 46.4 mm
- net /Block Diagram/LED PWM Connector/PWM_CH4_CONN: track 0.00 -> 31.7 mm
- net /Block Diagram/3V3 to 5V Logic Shifter/3V3_IO_3: track 16.0 -> 45.0 mm
- net /Block Diagram/MCU Enable and Boot/MCU_BOOT: track 2.62 -> 30.5 mm, vias 1 -> 2
- net /Block Diagram/3V3 to 5V Logic Shifter/3V3_IO_4: track 18.4 -> 46.2 mm
- net /Block Diagram/LED PWM Connector/PWM_CH3_CONN: track 0.00 -> 27.6 mm
- net /Block Diagram/MCU/GPIO_7_RS485_RX: track 0.00 -> 26.2 mm
- net /Block Diagram/3V3 to 5V Logic Shifter/5V_IO_3: track 0.00 -> 24.3 mm
- net /Block Diagram/3V3 to 5V Logic Shifter/5V_IO_2: track 0.00 -> 23.2 mm
- net /Block Diagram/LED PWM Connector/PWM_CH2_CONN: track 0.00 -> 22.9 mm
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- added copper zone on B.Cu, net +3V3
- added copper zone on F.Cu, net +3V3
- added copper zone on F.Cu, net +5V
- added copper zone on F.Cu, net +5V_IN
- added copper zone on F.Cu, net /Block Diagram/5V to 3.3V/SW_OUT
- added copper zone on F.Cu, net /Block Diagram/5V to 3.3V/SW_OUT_UNFILTERED
- added copper zone on F.Cu, net GND
