File: AstraControlPCB/power_connectors.kicad_sch (KiCad schematic)
At the start: 5 parts, among them CN1 4P JST VH

Commit message: Update wks file
Other:
- company: (none) -> LiveAstra Technologies
- title: Power Connectors -> AstraControl - Root
Changed lines of the file:
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@@
 	(paper "A4")
 	(title_block
-		(title "Power Connectors")
+		(title "AstraControl - Root")
+		(date "2024-08-26")
+		(rev "A")
+		(company "LiveAstra Technologies")
 	)
 	(junction

Commit message: workflow
Parts:
- added QST2, QST3: ~, symbol LiveAstra:Question_Box
Other:
- note added: "Power connectors"
Changed lines of the file:
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@@
+		)
+	)
+	(text "Power connectors"
+		(exclude_from_sim no)
+		(at 19.05 25.4 0)
+		(effects
+			(font
+				(face "ING Me Headline")
+				(size 8 8)
+			)
+			(justify left top)
 		)
 	)
@@
 		(dnp no)
 		(fields_autoplaced yes)
-		(property "Reference" "#FLG3"
+		(property "Reference" "#FLG03"
 			(at 218.44 76.835 0)
 			(effects
@@
 			(project "AstraControl"
 				(path "/9a751838-dce8-4d69-8a02-736625ac74e7/0db21d8e-3390-4d67-877f-0e5d98e37848/e0a60313-5e73-4a17-9374-b4b4ea2344cd"
-					(reference "#FLG3")
+					(reference "#FLG03")
 					(unit 1)
 				)
@@
 		(dnp no)
 		(fields_autoplaced yes)
-		(property "Reference" "#PWR34"
+		(property "Reference" "#PWR034"
 			(at 203.2 110.49 0)
 			(effects
@@
 			(project "AstraControl"
 				(path "/9a751838-dce8-4d69-8a02-736625ac74e7/0db21d8e-3390-4d67-877f-0e5d98e37848/e0a60313-5e73-4a17-9374-b4b4ea2344cd"
-					(reference "#PWR34")
+					(reference "#PWR034")
 					(unit 1)
 				)
@@
 	)
 	(symbol
+		(lib_id "LiveAstra:Question_Box")
+		(at 114.3 57.15 0)
+		(unit 1)
+		(exclude_from_sim yes)
+		(in_bom no)
+		(on_board no)
+		(dnp no)
+		(fields_autoplaced yes)
+		(property "Reference" "QST2"
+			(at 114.3 45.72 0)
+			(effects
+				(font
+					(size 1.27 1.27)
+				)
+			)
+		)
+		(property "Value" "~"
+			(at 114.3 48.26 0)
+			(effects
+				(font
+					(size 1.27 1.27)
+				)
+			)
+		)
+		(property "Footprint" ""
+			(at 99.822 53.34 0)
+			(effects
+				(font
+					(size 1.27 1.27)
+				)
+				(hide yes)
+			)
+		)
+		(property "Datasheet" ""
+			(at 99.822 53.34 0)
+			(effects
+				(font
+					(size 1.27 1.27)
+				)
+				(hide yes)
+			)
+		)
+		(property "Description" ""
+			(at 99.822 53.34 0)
+			(effects
+				(font
+					(size 1.27 1.27)
+				)
+				(hide yes)
+			)
+		)
+		(instances
+			(project ""
+				(path "/9a751838-dce8-4d69-8a02-736625ac74e7/0db21d8e-3390-4d67-877f-0e5d98e37848/e0a60313-5e73-4a17-9374-b4b4ea2344cd"
+					(reference "QST2")
+					(unit 1)
+				)
+			)
+		)
+	)
+	(symbol
 		(lib_id "LiveAstra:JST_VH_4PIN_10A_250V")
 		(at 71.12 83.82 180)
@@
 		(dnp no)
 		(fields_autoplaced yes)
-		(property "Reference" "#PWR35"
+		(property "Reference" "#PWR035"
 			(at 218.44 87.63 0)
 			(effects
@@
 			(project "AstraControl"
 				(path "/9a751838-dce8-4d69-8a02-736625ac74e7/0db21d8e-3390-4d67-877f-0e5d98e37848/e0a60313-5e73-4a17-9374-b4b4ea2344cd"
-					(reference "#PWR35")
+					(reference "#PWR035")
 					(unit 1)
 				)
@@
 		(dnp no)
 		(fields_autoplaced yes)
-		(property "Reference" "#PWR33"
+		(property "Reference" "#PWR033"
 			(at 203.2 86.36 0)
 			(effects
@@
 			(project "AstraControl"
 				(path "/9a751838-dce8-4d69-8a02-736625ac74e7/0db21d8e-3390-4d67-877f-0e5d98e37848/e0a60313-5e73-4a17-9374-b4b4ea2344cd"
-					(reference "#PWR33")
+					(reference "#PWR033")
+					(unit 1)
+				)
+			)
+		)
+	)
+	(symbol
+		(lib_name "Question_Box_1")
+		(lib_id "LiveAstra:Question_Box")
+		(at 171.45 57.15 0)
+		(unit 1)
+		(exclude_from_sim yes)
+		(in_bom no)
+		(on_board no)
+		(dnp no)
+		(fields_autoplaced yes)
+		(property "Reference" "QST3"
+			(at 171.45 45.72 0)
+			(effects
+				(font
+					(size 1.27 1.27)
+				)
+			)
+		)
+		(property "Value" "~"
+			(at 171.45 48.26 0)
+			(effects
+				(font
+					(size 1.27 1.27)
+				)
+			)
+		)
+		(property "Footprint" ""
+			(at 156.972 53.34 0)
+			(effects
+				(font
+					(size 1.27 1.27)
+				)
+				(hide yes)
+			)
+		)
+		(property "Datasheet" ""
+			(at 156.972 53.34 0)
+			(effects
+				(font
+					(size 1.27 1.27)
+				)
+				(hide yes)
+			)
+		)
+		(property "Description" ""
+			(at 156.972 53.34 0)
+			(effects
+				(font
+					(size 1.27 1.27)
+				)
+				(hide yes)
+			)
+		)
+		(instances
+			(project "AstraControl"
+				(path "/9a751838-dce8-4d69-8a02-736625ac74e7/0db21d8e-3390-4d67-877f-0e5d98e37848/e0a60313-5e73-4a17-9374-b4b4ea2344cd"
+					(reference "QST3")
 					(unit 1)
 				)
@@
 		(dnp no)
 		(fields_autoplaced yes)
-		(property "Reference" "#PWR30"
+		(property "Reference" "#PWR030"
 			(at 81.28 100.33 0)
 			(effects
@@
 			(project "AstraControl"
 				(path "/9a751838-dce8-4d69-8a02-736625ac74e7/0db21d8e-3390-4d67-877f-0e5d98e37848/e0a60313-5e73-4a17-9374-b4b4ea2344cd"
-					(reference "#PWR30")
+					(reference "#PWR030")
 					(unit 1)
 				)
@@
 		(dnp no)
 		(fields_autoplaced yes)
-		(property "Reference" "#PWR31"
+		(property "Reference" "#PWR031"
 			(at 101.6 107.95 0)
 			(effects
@@
 			(project "AstraControl"
 				(path "/9a751838-dce8-4d69-8a02-736625ac74e7/0db21d8e-3390-4d67-877f-0e5d98e37848/e0a60313-5e73-4a17-9374-b4b4ea2344cd"
-					(reference "#PWR31")
+					(reference "#PWR031")
 					(unit 1)
 				)
@@
 		(dnp no)
 		(fields_autoplaced yes)
-		(property "Reference" "#PWR36"
+		(property "Reference" "#PWR036"
 			(at 228.6 109.22 0)
 			(effects
@@
 			(project "AstraControl"
 				(path "/9a751838-dce8-4d69-8a02-736625ac74e7/0db21d8e-3390-4d67-877f-0e5d98e37848/e0a60313-5e73-4a17-9374-b4b4ea2344cd"
-					(reference "#PWR36")
+					(reference "#PWR036")
 					(unit 1)
 				)
@@
 		(dnp no)
 		(fields_autoplaced yes)
-		(property "Reference" "#FLG2"
+		(property "Reference" "#FLG02"
 			(at 203.2 76.835 0)
 			(effects
@@
 			(project "AstraControl"
 				(path "/9a751838-dce8-4d69-8a02-736625ac74e7/0db21d8e-3390-4d67-877f-0e5d98e37848/e0a60313-5e73-4a17-9374-b4b4ea2344cd"
-					(reference "#FLG2")
+					(reference "#FLG02")
 					(unit 1)
 				)
@@
 		(on_board yes)
 		(dnp no)
-		(property "Reference" "#FLG4"
+		(property "Reference" "#FLG04"
 			(at 233.68 76.835 0)
 			(effects
@@
 			(project "AstraControl"
 				(path "/9a751838-dce8-4d69-8a02-736625ac74e7/0db21d8e-3390-4d67-877f-0e5d98e37848/e0a60313-5e73-4a17-9374-b4b4ea2344cd"
-					(reference "#FLG4")
+					(reference "#FLG04")
 					(unit 1)
 				)
@@
 		(dnp no)
 		(fields_autoplaced yes)
-		(property "Reference" "#PWR32"
+		(property "Reference" "#PWR032"
 			(at 152.4 107.95 0)
 			(effects
@@
 			(project "AstraControl"
 				(path "/9a751838-dce8-4d69-8a02-736625ac74e7/0db21d8e-3390-4d67-877f-0e5d98e37848/e0a60313-5e73-4a17-9374-b4b4ea2344cd"
-					(reference "#PWR32")
-					(unit 1)
-				)
+					(reference "#PWR032")
+					(unit 1)
+				)

Commit message: update
Parts:
- renumbered TP11 to TP10, TP12 to TP11
Changed lines of the file:
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@@
 		(dnp no)
 		(fields_autoplaced yes)
-		(property "Reference" "TP11"
+		(property "Reference" "TP10"
 			(at 205.74 95.7876 0)
 			(effects
@@
 			(project ""
 				(path "/9a751838-dce8-4d69-8a02-736625ac74e7/0db21d8e-3390-4d67-877f-0e5d98e37848/e0a60313-5e73-4a17-9374-b4b4ea2344cd"
-					(reference "TP11")
+					(reference "TP10")
 					(unit 1)
 				)
@@
 		(dnp no)
 		(fields_autoplaced yes)
-		(property "Reference" "TP12"
+		(property "Reference" "TP11"
 			(at 231.14 95.7876 0)
 			(effects
@@
 			(project "AstraControl"
 				(path "/9a751838-dce8-4d69-8a02-736625ac74e7/0db21d8e-3390-4d67-877f-0e5d98e37848/e0a60313-5e73-4a17-9374-b4b4ea2344cd"
-					(reference "TP12")
-					(unit 1)
-				)
+					(reference "TP11")
+					(unit 1)
+				)

Commit message: update
Other:
- note added: "Are the TVS diodes enough or should I add anything extra? MOV / TBU?"
- note added: "Should there be another TVS between A and B?"
Changed lines of the file:
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@@
+		)
+	)
+	(text "Are the TVS diodes enough or should I add anything\nextra? MOV / TBU?"
+		(exclude_from_sim no)
+		(at 91.44 60.96 0)
+		(effects
+			(font
+				(face "ING Me")
+				(size 1.397 1.397)
+			)
+			(justify left)
+		)
+	)
+	(text "Should there be another TVS between A and B?"
+		(exclude_from_sim no)
+		(at 147.32 60.96 0)
+		(effects
+			(font
+				(face "ING Me")
+				(size 1.397 1.397)
+			)
+			(justify left)
 		)
 	)
@@
 	(symbol
 		(lib_id "LiveAstra:Question_Box")
-		(at 114.3 57.15 0)
+		(at 114.3 58.42 0)
 		(unit 1)
 		(exclude_from_sim yes)
@@
 		(fields_autoplaced yes)
 		(property "Reference" "QST2"
-			(at 114.3 45.72 0)
+			(at 114.3 46.99 0)
 			(effects
 				(font
@@
 		)
 		(property "Value" "~"
-			(at 114.3 48.26 0)
+			(at 114.3 49.53 0)
 			(effects
 				(font
@@
 		)
 		(property "Footprint" ""
-			(at 99.822 53.34 0)
+			(at 99.822 54.61 0)
 			(effects
 				(font
@@
 		)
 		(property "Datasheet" ""
-			(at 99.822 53.34 0)
+			(at 99.822 54.61 0)
 			(effects
 				(font
@@
 		)
 		(property "Description" ""
-			(at 99.822 53.34 0)
+			(at 99.822 54.61 0)
 			(effects
 				(font
@@
 	)
 	(symbol
-		(lib_name "Question_Box_1")
 		(lib_id "LiveAstra:Question_Box")
-		(at 171.45 57.15 0)
+		(at 170.18 58.42 0)
 		(unit 1)
 		(exclude_from_sim yes)
@@
 		(fields_autoplaced yes)
 		(property "Reference" "QST3"
-			(at 171.45 45.72 0)
+			(at 170.18 46.99 0)
 			(effects
 				(font
@@
 		)
 		(property "Value" "~"
-			(at 171.45 48.26 0)
+			(at 170.18 49.53 0)
 			(effects
 				(font
@@
 		)
 		(property "Footprint" ""
-			(at 156.972 53.34 0)
+			(at 155.702 54.61 0)
 			(effects
 				(font
@@
 		)
 		(property "Datasheet" ""
-			(at 156.972 53.34 0)
+			(at 155.702 54.61 0)
 			(effects
 				(font
@@
 		)
 		(property "Description" ""
-			(at 156.972 53.34 0)
-			(effects
-				(font
+			(at 155.702 54.61 0)
+			(effects
+				(font

Commit message: update
Other:
- note added: "Are the TVS diodes enough or should I add anything extra? MOV / TBU? Aiming to cover ~90% of cases."
- note added: "Should there be another TVS Diode between D- and D+?"
- note removed: "Are the TVS diodes enough or should I add anything extra? MOV / TBU?"
- note removed: "Should there be another TVS between A and B?"
Changed lines of the file:
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@@
 		)
 	)
-	(text "Are the TVS diodes enough or should I add anything\nextra? MOV / TBU?"
+	(text "Are the TVS diodes enough or should I add\nanything extra? MOV / TBU? \nAiming to cover ~90% of cases."
 		(exclude_from_sim no)
 		(at 91.44 60.96 0)
@@
 		)
 	)
-	(text "Should there be another TVS between A and B?"
+	(text "Should there be another TVS Diode \nbetween D- and D+?"
 		(exclude_from_sim no)
 		(at 147.32 60.96 0)

Commit message: Another redesign
Parts:
- added D1: SS14 Schottky, LiveAstra:D_SMA_SS14_C2480, symbol LiveAstra:D_Schottky_SS14_1A_40V
Connections:
- net 5V_IN: now also D1.1 (K)
- new net USB/VBUS: D1.2 (A)
Changed lines of the file:
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@@
+	(wire
+		(pts
+			(xy 132.08 119.38) (xy 152.4 119.38)
+		)
+		(stroke
+			(width 0)
+			(type default)
+		)
+	)
 	(wire
 		(pts
@@
 	(wire
 		(pts
-			(xy 76.2 119.38) (xy 101.6 119.38)
+			(xy 76.2 119.38) (xy 121.92 119.38)
 		)
 		(stroke
@@
 		)
 	)
-	(hierarchical_label "VBUS"
+	(hierarchical_label "5V_IN"
 		(shape output)
-		(at 101.6 119.38 0)
+		(at 81.28 76.2 0)
 		(fields_autoplaced yes)
 		(effects
@@
 		)
 	)
-	(hierarchical_label "5V_IN"
-		(shape output)
-		(at 81.28 76.2 0)
+	(hierarchical_label "USB_D+"
+		(shape bidirectional)
+		(at 101.6 124.46 0)
 		(fields_autoplaced yes)
 		(effects
@@
 		)
 	)
-	(hierarchical_label "USB_D+"
-		(shape bidirectional)
-		(at 101.6 124.46 0)
+	(hierarchical_label "5V_IN"
+		(shape output)
+		(at 152.4 119.38 0)
 		(fields_autoplaced yes)
 		(effects
@@
 					(unit 1)
 				)
+			)
+		)
+	)
+	(symbol
+		(lib_id "LiveAstra:D_Schottky_SS14_1A_40V")
+		(at 127 119.38 180)
+		(unit 1)
+		(exclude_from_sim no)
+		(in_bom yes)
+		(on_board yes)
+		(dnp no)
+		(fields_autoplaced yes)
+		(property "Reference" "D1"
+			(at 127.38 110.49 0)
+			(effects
+				(font
+					(size 1.27 1.27)
+				)
+			)
+		)
+		(property "Value" "SS14 Schottky"
+			(at 127.38 113.03 0)
+			(effects
+				(font
+					(size 1.27 1.27)
+					(bold yes)
+				)
+			)
+		)
+		(property "Footprint" "LiveAstra:D_SMA_SS14_C2480"
+			(at 127 110.49 0)
+			(effects
+				(font
+					(size 1.27 1.27)
+				)
+				(hide yes)
+			)
+		)
+		(property "Datasheet" "https://lcsc.com/product-detail/Schottky-Barrier-Diodes-SBD_SS14_C2480.html"
+			(at 127 106.68 0)
+			(effects
+				(font
+					(size 1.27 1.27)
+				)
+				(hide yes)
+			)
+		)
+		(property "Description" "Schottky Barrier Diode"
+			(at 127 114.3 0)
+			(effects
+				(font
+					(size 1.27 1.27)
+				)
+				(hide yes)
+			)
+		)
+		(property "LCSC Part" "C2480"
+			(at 127 102.87 0)
+			(effects
+				(font
+					(size 1.27 1.27)
+				)
+				(hide yes)
+			)
+		)
+		(property "Extra Values" "40V Single 1A 550mV@1A"
+			(at 127.38 115.57 0)
+			(effects
+				(font
+					(size 0.762 0.762)
+					(bold yes)
+				)
+			)
+		)
+		(pin "1"
+		)
+		(pin "2"
+		)
+		(instances
+			(project "AstraControl"
+				(path "/9a751838-dce8-4d69-8a02-736625ac74e7/0db21d8e-3390-4d67-877f-0e5d98e37848/e0a60313-5e73-4a17-9374-b4b4ea2344cd"
+					(reference "D1")
+					(unit 1)
+				)

Commit message: Updates
Parts:
- D2, D3: Extra Values 5A 50W 10V 5.6V Bidirectional -> 5A 50W 10V 5.6V 15pF Bidirectional
Changed lines of the file:
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@@
 			)
 		)
-		(property "Extra Values" "5A 50W 10V 5.6V Bidirectional"
+		(property "Extra Values" "5A 50W 10V 5.6V 15pF Bidirectional"
 			(at 105.41 96.5199 90)
 			(effects
@@
 			)
 		)
-		(property "Extra Values" "5A 50W 10V 5.6V Bidirectional"
+		(property "Extra Values" "5A 50W 10V 5.6V 15pF Bidirectional"
 			(at 156.21 96.5199 90)
 			(effects
