File: AstraControlPCB/5v_gpio_connectors.kicad_sch (KiCad schematic)
At the start: 2 parts, among them CN2 4P JST VH, CN3 4P JST VH

Commit message: Update wks file
Other:
- company: (none) -> LiveAstra Technologies
- title: 5V GPIO Connectors -> AstraControl - Root
Changed lines of the file:
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@@
 	(paper "A4")
 	(title_block
-		(title "5V GPIO Connectors")
+		(title "AstraControl - Root")
+		(date "2024-08-26")
+		(rev "A")
+		(company "LiveAstra Technologies")
 	)
 	(wire

Commit message: workflow
Other:
- note added: "5V GPIO Connectors"
Changed lines of the file:
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@@
+		)
+	)
+	(text "5V GPIO Connectors"
+		(exclude_from_sim no)
+		(at 19.05 25.4 0)
+		(effects
+			(font
+				(face "ING Me Headline")
+				(size 8 8)
+			)
+			(justify left top)
 		)
 	)
@@
 		(dnp no)
 		(fields_autoplaced yes)
-		(property "Reference" "#PWR52"
+		(property "Reference" "#PWR052"
 			(at 139.7 77.47 0)
 			(effects
@@
 			(project "AstraControl"
 				(path "/9a751838-dce8-4d69-8a02-736625ac74e7/0db21d8e-3390-4d67-877f-0e5d98e37848/a08072bc-5c98-487a-a9a6-bb737e215888"
-					(reference "#PWR52")
+					(reference "#PWR052")
 					(unit 1)
 				)
@@
 		(dnp no)
 		(fields_autoplaced yes)
-		(property "Reference" "#PWR51"
+		(property "Reference" "#PWR051"
 			(at 127 118.11 0)
 			(effects
@@
 			(project "AstraControl"
 				(path "/9a751838-dce8-4d69-8a02-736625ac74e7/0db21d8e-3390-4d67-877f-0e5d98e37848/a08072bc-5c98-487a-a9a6-bb737e215888"
-					(reference "#PWR51")
+					(reference "#PWR051")
 					(unit 1)
 				)
@@
 		(dnp no)
 		(fields_autoplaced yes)
-		(property "Reference" "#PWR50"
+		(property "Reference" "#PWR050"
 			(at 127 82.55 0)
 			(effects
@@
 			(project "AstraControl"
 				(path "/9a751838-dce8-4d69-8a02-736625ac74e7/0db21d8e-3390-4d67-877f-0e5d98e37848/a08072bc-5c98-487a-a9a6-bb737e215888"
-					(reference "#PWR50")
+					(reference "#PWR050")
 					(unit 1)
 				)
@@
 		(dnp no)
 		(fields_autoplaced yes)
-		(property "Reference" "#PWR53"
+		(property "Reference" "#PWR053"
 			(at 139.7 113.03 0)
 			(effects
@@
 			(project "AstraControl"
 				(path "/9a751838-dce8-4d69-8a02-736625ac74e7/0db21d8e-3390-4d67-877f-0e5d98e37848/a08072bc-5c98-487a-a9a6-bb737e215888"
-					(reference "#PWR53")
-					(unit 1)
-				)
+					(reference "#PWR053")
+					(unit 1)
+				)

Commit message: Silkscreen
Connections:
- net GPIO_35_5V is gone; now on net +5V_IN: CN2.3
- net GPIO_37_5V is gone; now on net +5V_IN: CN3.3
- net +5V_IN: no longer CN2.2, CN3.2
- net GND: now also CN2.2, CN3.2; no longer CN2.1, CN3.1
- net GPIO_36_5V renamed GPIO_41_5V
- net GPIO_38_5V renamed GPIO_39_5V
- new net GPIO_40_5V: CN3.1
- new net GPIO_42_5V: CN2.1

Commit message: Added MFN MPR to each components for eurocircuits
Parts:
- CN2, CN3: MFN (none) -> JST; MPN (none) -> B4P-VH(LF)(SN)
Changed lines of the file:
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@@
 			)
 		)
-		(property "Description" "VH CONNECTOR 3.96mm pitch/Disconnectable Crimp style connectors"
+		(property "Description" "1x4P 4P VH Tin 4 -25℃~+85℃ 10A 1 3.96mm Brass Direct Insert Plugin,P=3.96mm Wire To Board Connector ROHS"
 			(at 157.48 100.33 0)
 			(effects
@@
 					(bold yes)
 				)
+			)
+		)
+		(property "MFN" "JST"
+			(at 157.48 115.57 0)
+			(effects
+				(font
+					(size 1.27 1.27)
+				)
+				(hide yes)
+			)
+		)
+		(property "MPN" "B4P-VH(LF)(SN)"
+			(at 157.48 115.57 0)
+			(effects
+				(font
+					(size 1.27 1.27)
+				)
+				(hide yes)
 			)
 		)
@@
 			)
 		)
-		(property "Description" "VH CONNECTOR 3.96mm pitch/Disconnectable Crimp style connectors"
+		(property "Description" "1x4P 4P VH Tin 4 -25℃~+85℃ 10A 1 3.96mm Brass Direct Insert Plugin,P=3.96mm Wire To Board Connector ROHS"
 			(at 157.48 135.89 0)
 			(effects
@@
 			)
 		)
+		(property "MFN" "JST"
+			(at 157.48 151.13 0)
+			(effects
+				(font
+					(size 1.27 1.27)
+				)
+				(hide yes)
+			)
+		)
+		(property "MPN" "B4P-VH(LF)(SN)"
+			(at 157.48 151.13 0)
+			(effects
+				(font
+					(size 1.27 1.27)
+				)
+				(hide yes)
+			)
+		)

Commit message: Update schematic titles, templates
Other:
- title: AstraControl - Root -> AstraControl - 5V GPIO Connectors
Changed lines of the file:
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@@
 	(paper "A4")
 	(title_block
-		(title "AstraControl - Root")
+		(title "AstraControl - 5V GPIO Connectors")
 		(date "2024-08-26")
 		(rev "A")
